File: STM32F107RC.ETH.brd (EAGLE design)
At the start: 160 x 100 mm, 28 parts, among them J1 HR911105A, Q1 8MHz, U1 LAN8720A-CP, U2 STM32F107RCT6, X1 CB3LV-3I-74M2500

Commit message: Add files via upload
Parts:
- J2: device SparkFun-Connectors:LUXEON-PAD -> SparkFun-Connectors:1X01_OFFSET
- moved X1 48.8 mm to (106.7, 57.8), turned to 270 degrees
- moved R7 39.6 mm to (105.4, 63.8)
- moved R10 39.4 mm to (93.3, 57.5), turned to 90 degrees
- moved R6 34.0 mm to (100.3, 58.1), turned to 90 degrees
- moved R11 27.2 mm to (90.8, 57.5), turned to 90 degrees
- moved R8 25.0 mm to (83.2, 57.5)
- moved J1 19.5 mm to (94.6, 31.4)
- moved J2 18.4 mm to (108.3, 70.8), turned to 270 degrees
- moved C1 18.4 mm to (60.3, 83.2)
- moved C6 18.4 mm to (67.3, 73.0)
- moved C4 18.4 mm to (68.9, 40.0)
- moved R1 18.4 mm to (64.1, 45.4)
- moved C2 18.4 mm to (70.5, 55.6)
- moved C3 18.4 mm to (70.5, 53.0)
- moved JP2 18.4 mm to (39.4, 45.7)
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Connections:
- new net LED1: J1.10, U1.3
- new net LED2: J1.11, U1.2
- new net N$23: J1.1, U1.21
- new net N$28: J1.2, U1.20
- new net N$29: J1.3, U1.23
- new net N$31: J1.6, U1.22
- net N$10: now also J2.1; no longer J2.P$1
- net VCC: now also J1.12, J1.4, J1.5, J1.9, JP1.3

Commit message: Add files via upload
Parts:
- moved J1 4.97 mm to (92.4, 27.0), flipped to the bottom
Changed lines of the file:
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@@
 <attribute name="SPICEPREFIX" value="C" x="44.45" y="46.355" size="1.778" layer="27" rot="R90" display="off"/>
 </element>
-<element name="J1" library="HR911105A" package="HANRUN_HR911105A" value="HR911105A" x="94.615" y="31.4325" rot="R180">
-<attribute name="PACKAGE" value="None" x="94.615" y="31.4325" size="1.778" layer="27" rot="R180" display="off"/>
-<attribute name="MP" value="HR911105A" x="94.615" y="31.4325" size="1.778" layer="27" rot="R180" display="off"/>
-<attribute name="AVAILABILITY" value="Unavailable" x="94.615" y="31.4325" size="1.778" layer="27" rot="R180" display="off"/>
-<attribute name="PRICE" value="None" x="94.615" y="31.4325" size="1.778" layer="27" rot="R180" display="off"/>
-<attribute name="DESCRIPTION" value=" DIP RJ45 Connector; " x="94.615" y="31.4325" size="1.778" layer="27" rot="R180" display="off"/>
-<attribute name="MF" value="HanRun" x="94.615" y="31.4325" size="1.778" layer="27" rot="R180" display="off"/>
+<element name="J1" library="HR911105A" package="HANRUN_HR911105A" value="HR911105A" x="92.3925" y="26.9875" rot="MR180">
+<attribute name="PACKAGE" value="None" x="92.3925" y="26.9875" size="1.778" layer="28" rot="MR180" display="off"/>
+<attribute name="MP" value="HR911105A" x="92.3925" y="26.9875" size="1.778" layer="28" rot="MR180" display="off"/>
+<attribute name="AVAILABILITY" value="Unavailable" x="92.3925" y="26.9875" size="1.778" layer="28" rot="MR180" display="off"/>
+<attribute name="PRICE" value="None" x="92.3925" y="26.9875" size="1.778" layer="28" rot="MR180" display="off"/>
+<attribute name="DESCRIPTION" value=" DIP RJ45 Connector; " x="92.3925" y="26.9875" size="1.778" layer="28" rot="MR180" display="off"/>
+<attribute name="MF" value="HanRun" x="92.3925" y="26.9875" size="1.778" layer="28" rot="MR180" display="off"/>
 </element>
 <element name="J2" library="SparkFun-Connectors" package="1X01_OFFSET" value="" x="108.2675" y="70.8025" rot="R270"/>
@@
 <wire x1="44.45" y1="47.755" x2="104.58" y2="55.245" width="0" layer="19" extent="1-1"/>
 <wire x1="39.37" y1="46.99" x2="44.45" y2="47.755" width="0" layer="19" extent="1-1"/>
-<wire x1="99.055" y1="40.3225" x2="73.66" y2="42.2275" width="0" layer="19" extent="1-1"/>
+<wire x1="87.9525" y1="35.8775" x2="73.66" y2="42.2275" width="0" layer="19" extent="1-1"/>
 </signal>
 <signal name="N$6">
@@
 <contactref element="J1" pad="12"/>
 <wire x1="90.7375" y1="49.2425" x2="108.78" y2="60.325" width="0" layer="19" extent="1-1"/>
-<wire x1="93.975" y1="40.3225" x2="90.7375" y2="49.2425" width="0" layer="19" extent="1-1"/>
-<wire x1="95.245" y1="37.7825" x2="93.975" y2="40.3225" width="0" layer="19" extent="1-1"/>
-<wire x1="101.24" y1="26.5325" x2="95.245" y2="37.7825" width="0" layer="19" extent="1-1"/>
-<wire x1="87.99" y1="26.5325" x2="101.24" y2="26.5325" width="0" layer="19" extent="1-1"/>
+<wire x1="93.0325" y1="35.8775" x2="90.7375" y2="49.2425" width="0" layer="19" extent="1-1"/>
+<wire x1="91.7625" y1="33.3375" x2="93.0325" y2="35.8775" width="0" layer="19" extent="1-1"/>
+<wire x1="85.7675" y1="22.0875" x2="91.7625" y2="33.3375" width="0" layer="19" extent="1-1"/>
+<wire x1="99.0175" y1="22.0875" x2="85.7675" y2="22.0875" width="0" layer="19" extent="1-1"/>
 <wire x1="60.325" y1="48.5775" x2="90.7375" y2="49.2425" width="0" layer="19" extent="1-1"/>
 <wire x1="60.325" y1="51.7525" x2="60.325" y2="48.5775" width="0" layer="19" extent="1-1"/>
@@
 <contactref element="U1" pad="21"/>
 <contactref element="J1" pad="1"/>
-<wire x1="90.165" y1="37.7825" x2="90.2375" y2="45.3725" width="0" layer="19" extent="1-1"/>
+<wire x1="96.8425" y1="33.3375" x2="90.2375" y2="45.3725" width="0" layer="19" extent="1-1"/>
 </signal>
 <signal name="N$28">
 <contactref element="U1" pad="20"/>
 <contactref element="J1" pad="2"/>
-<wire x1="91.435" y1="40.3225" x2="89.7375" y2="45.3725" width="0" layer="19" extent="1-1"/>
+<wire x1="95.5725" y1="35.8775" x2="89.7375" y2="45.3725" width="0" layer="19" extent="1-1"/>
 </signal>
 <signal name="N$29">
 <contactref element="U1" pad="23"/>
 <contactref element="J1" pad="3"/>
-<wire x1="92.705" y1="37.7825" x2="91.2375" y2="45.3725" width="0" layer="19" extent="1-1"/>
+<wire x1="94.3025" y1="33.3375" x2="91.2375" y2="45.3725" width="0" layer="19" extent="1-1"/>
 </signal>
 <signal name="N$31">
 <contactref element="U1" pad="22"/>
 <contactref element="J1" pad="6"/>
-<wire x1="96.515" y1="40.3225" x2="90.7375" y2="45.3725" width="0" layer="19" extent="1-1"/>
+<wire x1="90.4925" y1="35.8775" x2="90.7375" y2="45.3725" width="0" layer="19" extent="1-1"/>
 </signal>
 <signal name="LED2">
 <contactref element="U1" pad="2"/>
 <contactref element="J1" pad="11"/>
-<wire x1="98.7" y1="26.5325" x2="92.4225" y2="46.5575" width="0" layer="19" extent="1-1"/>
+<wire x1="88.3075" y1="22.0875" x2="92.4225" y2="46.5575" width="0" layer="19" extent="1-1"/>
 </signal>
 <signal name="LED1">
 <contactref element="U1" pad="3"/>
 <contactref element="J1" pad="10"/>
-<wire x1="90.53" y1="26.5325" x2="92.4225" y2="47.0575" width="0" layer="19" extent="1-1"/>
+<wire x1="96.4775" y1="22.0875" x2="92.4225" y2="47.0575" width="0" layer="19" extent="1-1"/>
 </signal>
 </signals>

Commit message: Add files via upload
Parts:
- added R13, R14: 330R, resistor:0204/7
- moved C3 37.5 mm to (108.0, 51.4), turned to 90 degrees
- moved C2 33.6 mm to (103.8, 51.4), turned to 90 degrees
- moved R9 16.6 mm to (88.6, 57.5), turned to 90 degrees
- moved R1 16.3 mm to (79.7, 50.2)
- moved J1 4.97 mm to (94.6, 31.4), flipped to the top
- moved R10 0.32 mm to (93.0, 57.5)
Connections:
- new net SIG_LED01: R14.2, U1.3
- new net SIG_LED02: R13.2, U1.2
- net LED1: now also R14.1; no longer U1.3
- net LED2: now also R13.1; no longer U1.2
- net N$4: now also U2.23

Commit message: Add files via upload
Parts:
- R5: value 12.1K -> 4K7
Connections:
- removed net N$11: L1.1, U1.1, U1.19
- new net AVDD: J1.4, J1.5, L1.1, U1.1, U1.19
- net VCC: no longer J1.4, J1.5
Changed lines of the file:
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@@
 <attribute name="SPICEPREFIX" value="R" x="77.47" y="42.2275" size="1.778" layer="27" display="off"/>
 </element>
-<element name="R5" library="resistor" package="0204/7" value="12.1K" x="60.6425" y="36.83" rot="R90">
+<element name="R5" library="resistor" package="0204/7" value="4K7" x="60.6425" y="36.83" rot="R90">
 <attribute name="SPICEPREFIX" value="R" x="60.6425" y="36.83" size="1.778" layer="27" rot="R90" display="off"/>
 </element>
@@
 <wire x1="108.2675" y1="70.8025" x2="95.84" y2="70.735" width="0" layer="19" extent="1-1"/>
 </signal>
-<signal name="N$11">
+<signal name="AVDD">
 <contactref element="U1" pad="19"/>
 <contactref element="U1" pad="1"/>
 <contactref element="L1" pad="1"/>
-<wire x1="92.4225" y1="46.0575" x2="89.2375" y2="45.3725" width="0" layer="19" extent="1-1"/>
-<wire x1="67.945" y1="51.7525" x2="92.4225" y2="46.0575" width="0" layer="19" extent="1-1"/>
+<contactref element="J1" pad="4"/>
+<contactref element="J1" pad="5"/>
+<wire x1="89.2375" y1="45.3725" x2="92.4225" y2="46.0575" width="0" layer="19" extent="1-1"/>
+<wire x1="93.975" y1="40.3225" x2="92.4225" y2="46.0575" width="0" layer="19" extent="1-1"/>
+<wire x1="95.245" y1="37.7825" x2="93.975" y2="40.3225" width="0" layer="19" extent="1-1"/>
+<wire x1="67.945" y1="51.7525" x2="89.2375" y2="45.3725" width="0" layer="19" extent="1-1"/>
 </signal>
 <signal name="N$12">
@@
 <contactref element="C7" pad="1"/>
 <contactref element="JP1" pad="3"/>
-<contactref element="J1" pad="4"/>
-<contactref element="J1" pad="5"/>
 <contactref element="J1" pad="9"/>
 <contactref element="J1" pad="12"/>
 <wire x1="90.7375" y1="49.2425" x2="108.78" y2="60.325" width="0" layer="19" extent="1-1"/>
-<wire x1="93.975" y1="40.3225" x2="90.7375" y2="49.2425" width="0" layer="19" extent="1-1"/>
-<wire x1="95.245" y1="37.7825" x2="93.975" y2="40.3225" width="0" layer="19" extent="1-1"/>
-<wire x1="101.24" y1="26.5325" x2="95.245" y2="37.7825" width="0" layer="19" extent="1-1"/>
-<wire x1="87.99" y1="26.5325" x2="101.24" y2="26.5325" width="0" layer="19" extent="1-1"/>
-<wire x1="60.325" y1="48.5775" x2="90.7375" y2="49.2425" width="0" layer="19" extent="1-1"/>
-<wire x1="60.325" y1="51.7525" x2="60.325" y2="48.5775" width="0" layer="19" extent="1-1"/>
-<wire x1="75.8825" y1="50.165" x2="60.325" y2="48.5775" width="0" layer="19" extent="1-1"/>
-<wire x1="60.6425" y1="40.64" x2="75.8825" y2="50.165" width="0" layer="19" extent="1-1"/>
-<wire x1="44.45" y1="44.955" x2="75.8825" y2="50.165" width="0" layer="19" extent="1-1"/>
+<wire x1="75.8825" y1="50.165" x2="90.7375" y2="49.2425" width="0" layer="19" extent="1-1"/>
+<wire x1="60.325" y1="51.7525" x2="75.8825" y2="50.165" width="0" layer="19" extent="1-1"/>
+<wire x1="60.325" y1="48.5775" x2="60.325" y2="51.7525" width="0" layer="19" extent="1-1"/>
+<wire x1="60.6425" y1="40.64" x2="60.325" y2="48.5775" width="0" layer="19" extent="1-1"/>
+<wire x1="44.45" y1="44.955" x2="60.325" y2="48.5775" width="0" layer="19" extent="1-1"/>
 <wire x1="39.37" y1="44.45" x2="44.45" y2="44.955" width="0" layer="19" extent="1-1"/>
+<wire x1="87.99" y1="26.5325" x2="90.7375" y2="49.2425" width="0" layer="19" extent="1-1"/>
+<wire x1="101.24" y1="26.5325" x2="87.99" y2="26.5325" width="0" layer="19" extent="1-1"/>
 <wire x1="55.245" y1="76.835" x2="60.325" y2="51.7525" width="0" layer="19" extent="1-1"/>
 <wire x1="79.6925" y1="87.3125" x2="55.245" y2="76.835" width="0" layer="19" extent="1-1"/>

Commit message: Add files via upload
Parts:
- added C8: 222, resistor:C1206
Connections:
- net N$23 renamed TD+
- net N$28 renamed TD-
- net N$29 renamed RD+
- net N$31 renamed RD-
- net AVDD: now also C8.1
- net GND: now also C8.2
Changed lines of the file:
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@@
 <attribute name="SPICEPREFIX" value="R" x="5.08" y="-8.89" size="1.778" layer="27" display="off"/>
+</element>
+<element name="C8" library="resistor" package="C1206" value="222" x="2.54" y="-13.0175">
+<attribute name="SPICEPREFIX" value="C" x="2.54" y="-13.0175" size="1.778" layer="27" display="off"/>
 </element>
 </elements>
@@
 <contactref element="J1" pad="4"/>
 <contactref element="J1" pad="5"/>
+<contactref element="C8" pad="1"/>
 <wire x1="89.2375" y1="45.3725" x2="92.4225" y2="46.0575" width="0" layer="19" extent="1-1"/>
 <wire x1="93.975" y1="40.3225" x2="92.4225" y2="46.0575" width="0" layer="19" extent="1-1"/>
 <wire x1="95.245" y1="37.7825" x2="93.975" y2="40.3225" width="0" layer="19" extent="1-1"/>
 <wire x1="67.945" y1="51.7525" x2="89.2375" y2="45.3725" width="0" layer="19" extent="1-1"/>
+<wire x1="1.14" y1="-13.0175" x2="67.945" y2="51.7525" width="0" layer="19" extent="1-1"/>
 </signal>
 <signal name="N$12">
@@
 <contactref element="C7" pad="2"/>
 <contactref element="J1" pad="8"/>
+<contactref element="C8" pad="2"/>
 <wire x1="65.91" y1="73.025" x2="79.6925" y2="82.2325" width="0" layer="19" extent="1-1"/>
 <wire x1="65.91" y1="67.945" x2="65.91" y2="73.025" width="0" layer="19" extent="1-1"/>
 <wire x1="60.325" y1="81.785" x2="65.91" y2="73.025" width="0" layer="19" extent="1-1"/>
-<wire x1="104.58" y1="55.245" x2="65.91" y2="67.945" width="0" layer="19" extent="1-1"/>
-<wire x1="103.8225" y1="52.835" x2="104.58" y2="55.245" width="0" layer="19" extent="1-1"/>
-<wire x1="107.95" y1="52.835" x2="103.8225" y2="52.835" width="0" layer="19" extent="1-1"/>
-<wire x1="68.8975" y1="41.405" x2="107.95" y2="52.835" width="0" layer="19" extent="1-1"/>
+<wire x1="68.8975" y1="41.405" x2="65.91" y2="67.945" width="0" layer="19" extent="1-1"/>
 <wire x1="73.66" y1="42.2275" x2="68.8975" y2="41.405" width="0" layer="19" extent="1-1"/>
-<wire x1="44.45" y1="47.755" x2="104.58" y2="55.245" width="0" layer="19" extent="1-1"/>
+<wire x1="44.45" y1="47.755" x2="68.8975" y2="41.405" width="0" layer="19" extent="1-1"/>
 <wire x1="39.37" y1="46.99" x2="44.45" y2="47.755" width="0" layer="19" extent="1-1"/>
 <wire x1="99.055" y1="40.3225" x2="73.66" y2="42.2275" width="0" layer="19" extent="1-1"/>
+<wire x1="103.8225" y1="52.835" x2="99.055" y2="40.3225" width="0" layer="19" extent="1-1"/>
+<wire x1="104.58" y1="55.245" x2="103.8225" y2="52.835" width="0" layer="19" extent="1-1"/>
+<wire x1="107.95" y1="52.835" x2="103.8225" y2="52.835" width="0" layer="19" extent="1-1"/>
+<wire x1="3.94" y1="-13.0175" x2="39.37" y2="46.99" width="0" layer="19" extent="1-1"/>
 </signal>
 <signal name="N$6">
@@
 <wire x1="68.71" y1="67.945" x2="73.66" y2="68.072" width="0" layer="19" extent="1-1"/>
 </signal>
-<signal name="N$23">
+<signal name="TD+">
 <contactref element="U1" pad="21"/>
 <contactref element="J1" pad="1"/>
 <wire x1="90.165" y1="37.7825" x2="90.2375" y2="45.3725" width="0" layer="19" extent="1-1"/>
 </signal>
-<signal name="N$28">
+<signal name="TD-">
 <contactref element="U1" pad="20"/>
 <contactref element="J1" pad="2"/>
 <wire x1="91.435" y1="40.3225" x2="89.7375" y2="45.3725" width="0" layer="19" extent="1-1"/>
 </signal>
-<signal name="N$29">
+<signal name="RD+">
 <contactref element="U1" pad="23"/>
 <contactref element="J1" pad="3"/>
 <wire x1="92.705" y1="37.7825" x2="91.2375" y2="45.3725" width="0" layer="19" extent="1-1"/>
 </signal>
-<signal name="N$31">
+<signal name="RD-">
 <contactref element="U1" pad="22"/>
 <contactref element="J1" pad="6"/>

Commit message: Add files via upload
Parts:
- added R15, R16, R17, R18: 1k, resistor:0204/7
- moved J1 14.9 mm to (90.5, 17.1)
- moved U1 2.48 mm to (90.2, 44.8)
- moved C2 0.63 mm to (104.5, 51.4)
Connections:
- net AVDD: now also R15.2, R16.2, R17.2, R18.2
- net RD+: now also R17.1
- net RD-: now also R18.1
- net TD+: now also R15.1
- net TD-: now also R16.1
Routing:
- net TD+: track 0.00 -> 34.3 mm, vias 0 -> 2
- net RD+: track 0.00 -> 26.5 mm, vias 0 -> 1
- net AVDD: track 0.00 -> 25.7 mm
- net RD-: track 0.00 -> 24.9 mm
- net TD-: track 0.00 -> 24.4 mm

Commit message: Add files via upload
Parts:
- moved R14 101.3 mm to (97.7, 32.2), turned to 180 degrees
- moved R13 98.6 mm to (97.7, 30.0), turned to 180 degrees
- moved C8 75.2 mm to (42.4, 50.7), turned to 180 degrees
- moved U2 2.56 mm to (90.5, 73.0)
Routing:
- net SIG_LED02: track 0.00 -> 16.6 mm
- net SIG_LED01: track 0.00 -> 14.0 mm

Commit message: Add files via upload
Parts:
- moved X1 14.7 mm to (92.3, 54.5), turned to 90 degrees
- moved R1 9.86 mm to (87.8, 55.8), turned to 270 degrees
- moved R9 9.37 mm to (79.2, 57.2)
- moved R11 7.54 mm to (98.3, 57.2)
- moved R10 7.46 mm to (100.5, 57.3)
- moved R8 6.04 mm to (77.2, 57.2)
- moved C2 2.98 mm to (103.0, 48.8)
- moved C3 2.79 mm to (108.7, 48.7)
- moved R6 2.54 mm to (102.7, 57.2)
Routing:
- net N$7: track 0.00 -> 17.5 mm
- net N$8: track 0.00 -> 16.3 mm, vias 0 -> 2
- net N$19: track 0.00 -> 2.69 mm
