File: STM32F107RC.ETH.brd (EAGLE design)
At the start: 160 x 100 mm, 35 parts, among them J1 HR911105A, Q1 8MHz, U1 LAN8720A-CP, U2 STM32F107RCT6, X1 CB3LV-3I-74M2500

Commit message: desktop update
Parts:
- moved R4 21.4 mm to (97.7, 35.4), turned to 180 degrees
Routing:
- net SIG_LED02: track 16.6 -> 19.0 mm
- net SIG_LED01: track 14.0 -> 16.1 mm
Changed lines of the file:
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@@
 <attribute name="SPICEPREFIX" value="R" x="55.245" y="80.645" size="1.778" layer="27" rot="R270" display="off"/>
 </element>
-<element name="R4" library="resistor" package="0204/7" value="12.1K" x="77.47" y="42.2275">
-<attribute name="SPICEPREFIX" value="R" x="77.47" y="42.2275" size="1.778" layer="27" display="off"/>
+<element name="R4" library="resistor" package="0204/7" value="12.1K" x="97.710625" y="35.40125" rot="R180">
+<attribute name="SPICEPREFIX" value="R" x="97.710625" y="35.40125" size="1.778" layer="27" rot="R180" display="off"/>
 </element>
 <element name="R5" library="resistor" package="0204/7" value="4K7" x="60.6425" y="36.83" rot="R90">
@@
 <wire x1="60.325" y1="81.785" x2="65.91" y2="73.025" width="0" layer="19" extent="1-1"/>
 <wire x1="68.8975" y1="41.405" x2="65.91" y2="67.945" width="0" layer="19" extent="1-1"/>
-<wire x1="73.66" y1="42.2275" x2="68.8975" y2="41.405" width="0" layer="19" extent="1-1"/>
-<wire x1="94.413125" y1="57.070625" x2="73.66" y2="42.2275" width="0" layer="19" extent="1-1"/>
+<wire x1="101.520625" y1="35.40125" x2="68.8975" y2="41.405" width="0" layer="19" extent="1-1"/>
+<wire x1="94.413125" y1="57.070625" x2="101.520625" y2="35.40125" width="0" layer="19" extent="1-1"/>
 <wire x1="103.02875" y1="50.215625" x2="94.413125" y2="57.070625" width="0" layer="19" extent="1-1"/>
 <wire x1="108.664375" y1="50.13625" x2="103.02875" y2="50.215625" width="0" layer="19" extent="1-1"/>
@@
 <wire x1="40.98625" y1="50.720625" x2="44.45" y2="47.755" width="0" layer="19" extent="1-1"/>
 <wire x1="39.37" y1="46.99" x2="40.98625" y2="50.720625" width="0" layer="19" extent="1-1"/>
-<wire x1="94.9275" y1="26.035" x2="73.66" y2="42.2275" width="0" layer="19" extent="1-1"/>
+<wire x1="94.9275" y1="26.035" x2="101.520625" y2="35.40125" width="0" layer="19" extent="1-1"/>
 </signal>
 <signal name="N$6">
@@
 <contactref element="U1" pad="24"/>
 <contactref element="R4" pad="2"/>
-<wire x1="81.28" y1="42.2275" x2="91.42" y2="42.911875" width="0" layer="19" extent="1-1"/>
+<wire x1="93.900625" y1="35.40125" x2="91.42" y2="42.911875" width="0" layer="19" extent="1-1"/>
 </signal>
 <signal name="N$20">
@@
 <wire x1="92.105" y1="44.096875" x2="93.1425" y2="44.096875" width="0.3048" layer="1"/>
 <wire x1="93.1425" y1="44.096875" x2="93.345" y2="43.894375" width="0.3048" layer="1"/>
-<wire x1="93.345" y1="43.894375" x2="93.345" y2="33.734375" width="0.3048" layer="1"/>
 <wire x1="93.345" y1="33.734375" x2="92.313125" y2="32.7025" width="0.3048" layer="1"/>
 <wire x1="92.313125" y1="32.7025" x2="92.313125" y2="31.115" width="0.3048" layer="1"/>
@@
 <wire x1="93.0275" y1="30.400625" x2="93.50375" y2="30.400625" width="0.3048" layer="1"/>
 <wire x1="93.50375" y1="30.400625" x2="93.900625" y2="30.00375" width="0.3048" layer="1"/>
+<wire x1="93.345" y1="43.894375" x2="93.345" y2="39.37" width="0.3048" layer="1"/>
+<wire x1="93.345" y1="39.37" x2="95.488125" y2="37.226875" width="0.3048" layer="1"/>
+<wire x1="95.488125" y1="37.226875" x2="95.488125" y2="34.845625" width="0.3048" layer="1"/>
+<wire x1="95.488125" y1="34.845625" x2="94.376875" y2="33.734375" width="0.3048" layer="1"/>
+<wire x1="94.376875" y1="33.734375" x2="93.345" y2="33.734375" width="0.3048" layer="1"/>
 </signal>
 <signal name="SIG_LED01">
 <contactref element="U1" pad="3"/>
 <contactref element="R14" pad="2"/>
-<wire x1="93.900625" y1="32.22625" x2="93.900625" y2="43.02125" width="0.4064" layer="1"/>
 <wire x1="93.900625" y1="43.02125" x2="93.900625" y2="44.370625" width="0.3048" layer="1"/>
 <wire x1="92.116875" y1="44.60875" x2="93.6625" y2="44.60875" width="0.3048" layer="1"/>
 <wire x1="93.6625" y1="44.60875" x2="93.900625" y2="44.370625" width="0.3048" layer="1"/>
 <wire x1="92.116875" y1="44.60875" x2="92.105" y2="44.596875" width="0" layer="19" extent="1-1"/>
+<wire x1="93.900625" y1="43.02125" x2="93.900625" y2="39.766875" width="0.4064" layer="1"/>
+<wire x1="93.900625" y1="39.766875" x2="96.36125" y2="37.30625" width="0.4064" layer="1"/>
+<wire x1="96.36125" y1="37.30625" x2="96.36125" y2="34.686875" width="0.4064" layer="1"/>
+<wire x1="96.36125" y1="34.686875" x2="93.900625" y2="32.22625" width="0.4064" layer="1"/>
 </signal>
 </signals>

Commit message: u from surface
Parts:
- moved C4 31.0 mm to (99.8, 37.9), turned to 0 degrees
- moved R7 6.59 mm to (105.2, 57.2), turned to 270 degrees
- moved C3 4.95 mm to (103.8, 47.7)
- moved C2 4.25 mm to (98.9, 47.8)
- moved R1 1.14 mm to (88.3, 54.8)
- moved X1 1.14 mm to (92.8, 53.5)
Routing:
- net N$13: track 0.00 -> 8.54 mm

Commit message: u g
Parts:
- moved C4 19.2 mm to (81.4, 43.6), turned to 270 degrees
- moved R5 17.0 mm to (75.4, 45.2), turned to 180 degrees
- moved JP1 4.51 mm to (76.0, 87.3)
- moved R12 3.83 mm to (84.5, 87.9)
- moved C3 2.89 mm to (105.3, 45.2), turned to 270 degrees
- moved C2 2.54 mm to (98.7, 45.2), turned to 270 degrees
- moved R1 0.58 mm to (87.7, 54.9)
Connections:
- removed net VSS: U1.25
- net GND: now also U1.25
- net N$16: now also U1.15
Routing:
- net GND: track 0.00 -> 16.6 mm, vias 0 -> 2
- net N$14: track 0.00 -> 13.5 mm
- net AVDD: track 32.4 -> 41.9 mm, vias 0 -> 2
- net N$16: track 0.00 -> 9.37 mm
- net N$7: track 17.5 -> 11.8 mm
- net N$19: track 2.69 -> 3.57 mm
- net SIG_LED01: track 16.1 -> 16.7 mm
- net SIG_LED02: track 19.0 -> 19.6 mm

Commit message: lenovo up
Parts:
- moved C8 31.0 mm to (71.5, 40.1)
- moved L1 16.9 mm to (71.4, 36.5)
- moved JP1 7.93 mm to (68.7, 84.2)
- moved C5 4.62 mm to (70.2, 71.5)
- moved Q1 4.62 mm to (76.6, 74.1)
- moved C6 4.62 mm to (70.2, 76.6)
- moved R12 3.74 mm to (84.8, 84.2)
- moved J2 2.49 mm to (108.7, 73.3)
Routing:
- net N$27: track 0.00 -> 14.8 mm
- net N$26: track 0.00 -> 13.8 mm
- net AVDD: track 41.9 -> 55.1 mm
- net N$10: track 0.00 -> 12.5 mm
- net N$24: track 0.00 -> 12.3 mm
- net GND: track 16.6 -> 26.8 mm
- net N$25: track 0.00 -> 5.59 mm

Commit message: 5.11.18
Parts:
- moved C7 22.7 mm to (66.7, 41.9), turned to 270 degrees
- moved JP2 22.1 mm to (61.2, 42.1), turned to 180 degrees
- moved R3 21.1 mm to (70.6, 66.1), turned to 180 degrees
- moved R2 20.4 mm to (84.5, 50.6)
- moved C1 17.7 mm to (70.2, 68.6), turned to 180 degrees
- moved R1 8.11 mm to (79.9, 57.2)
- moved L1 5.08 mm to (73.9, 41.0)
- moved J1 3.57 mm to (90.6, 13.6), flipped to the bottom
- moved C8 2.56 mm to (72.2, 37.6)
- moved R8 2.47 mm to (74.7, 57.1)
- moved R9 1.99 mm to (77.2, 57.1)
- moved R7 0.95 mm to (106.1, 57.2)
- moved X1 0.48 mm to (92.8, 54.0)
Connections:
- removed net VBAT: U2.1
- removed net VDDA: U2.13
- removed net VDD_1: U2.32
- removed net VDD_2: U2.48
- removed net VDD_3: U2.64
- removed net VDD_4: U2.19
- removed net VSSA: U2.12
- removed net VSS_1: U2.31
- removed net VSS_2: U2.47
- removed net VSS_3: U2.63
- removed net VSS_4: U2.18
- net GND: now also U2.12, U2.18, U2.31, U2.47, U2.63
- net VCC: now also U2.1, U2.13, U2.19, U2.32, U2.48, U2.64
Routing:
- net VCC: track 0.00 -> 100.9 mm, vias 0 -> 2
- net GND: track 26.8 -> 122.8 mm
- net N$9: track 0.00 -> 69.3 mm, vias 0 -> 2
- net N$2: track 0.00 -> 35.2 mm, vias 0 -> 4
- net N$17: track 0.00 -> 27.2 mm
- net N$1: track 0.00 -> 25.9 mm, vias 0 -> 2
- net N$8: track 16.6 -> 42.0 mm, vias 2 -> 3
- net N$18: track 0.00 -> 22.3 mm
- net N$4: track 0.00 -> 21.5 mm
- net N$20: track 0.00 -> 19.7 mm
- net N$6: track 0.00 -> 18.8 mm
- net N$7: track 11.8 -> 30.5 mm, vias 0 -> 3
- net N$15: track 0.00 -> 16.2 mm
- net N$19: track 3.57 -> 17.8 mm
- net N$5: track 0.00 -> 14.1 mm
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
Commit message: 6.11.18
Parts:
- added C10, C9: 104, resistor:C1206
- moved R14 1.83 mm to (97.7, 34.1)
- moved R4 1.83 mm to (97.7, 37.2)
- moved R13 1.83 mm to (97.7, 31.8)
- moved Q1 1.27 mm to (75.3, 74.1)
Connections:
- net GND: now also C10.2, C9.2
- net VCC: now also C10.1, C9.1
Routing:
- net GND: track 122.8 -> 197.4 mm, vias 2 -> 6
- net VCC: track 100.9 -> 131.5 mm, vias 2 -> 4
- net RD+: track 14.3 -> 39.1 mm
- net TD+: track 27.2 -> 46.0 mm
- net TD-: track 17.0 -> 32.8 mm, vias 0 -> 2
- net AVDD: track 45.1 -> 59.2 mm
- net RD-: track 11.4 -> 25.5 mm, vias 0 -> 2
- net SIG_LED02: track 20.4 -> 14.2 mm
- net SIG_LED01: track 16.5 -> 11.1 mm
- net N$13: track 8.54 -> 5.03 mm
- net N$6: track 18.8 -> 21.1 mm
- net N$26: track 13.8 -> 14.4 mm

Commit message: u 6.11.18
Parts:
- added C11: 105, resistor:C1206
- added J3: USB-MICROB, SparkFun-Connectors:USB-MICROB
- added J4: (no value), SparkFun-Connectors:1X05_LOCK_LONGPADS
- added JP3: (no value), jumper:JP1
- added U3: LM1117MP-3.3, LM1117MP-3.3:SOT230P696X180-4N
- added X2: MSTBA6, con-phoenix-508:MSTBA6
Connections:
- new net N$23: C11.1, JP3.1, U3.3
- net GND: now also C11.2, JP3.2, U3.1
- net VCC: now also U3.4
Routing:
- net LED1: track 0.00 -> 35.9 mm
- net LED2: track 0.00 -> 35.7 mm
- net SIG_LED01: track 11.1 -> 14.2 mm
- net SIG_LED02: track 14.2 -> 17.1 mm
- net AVDD: track 59.2 -> 56.9 mm
- net N$19: track 17.8 -> 19.9 mm
- net N$20: track 19.7 -> 21.0 mm
- net N$26: track 14.4 -> 13.8 mm

Commit message: u 9-11-18
Parts:
- removed J4: (no value), SparkFun-Connectors:1X05_LOCK_LONGPADS
- added J5: (no value), SparkFun-Connectors:MOLEX-1X6
- moved X2 28.8 mm to (25.6, 52.1)
- moved J3 16.3 mm to (23.5, 27.1)
Connections:
- removed net N$6: C1.1, R3.1, U2.7
- new net N$11: J5.1, U2.55
- new net NRST: C1.1, J5.5, R3.1, U2.7
- new net SWCLK: J5.4, U2.49
- new net SWDIO: J5.3, U2.46
- net GND: now also J5.6
- net VCC: now also J5.2
Routing:
- net NRST: track 0.00 -> 21.1 mm
- net N$6: track 21.1 -> 0.00 mm
- net SWCLK: track 0.00 -> 5.39 mm
- net SWDIO: track 0.00 -> 4.44 mm
Changed lines of the file:
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@@
 <attribute name="SPICEPREFIX" value="C" x="69.85" y="21.034375" size="1.778" layer="27" rot="R180" display="off"/>
 </element>
-<element name="X2" library="con-phoenix-508" package="MSTBA6" value="MSTBA6" x="26.035" y="80.883125" rot="R270">
-<attribute name="OC_NEWARK" value="71C4165" x="26.035" y="80.883125" size="1.778" layer="27" rot="R270" display="off"/>
-<attribute name="MPN" value="1757284" x="26.035" y="80.883125" size="1.778" layer="27" rot="R270" display="off"/>
-<attribute name="MF" value="FARNELL" x="26.035" y="80.883125" size="1.778" layer="27" rot="R270" display="off"/>
-<attribute name="OC_FARNELL" value="3705213" x="26.035" y="80.883125" size="1.778" layer="27" rot="R270" display="off"/>
+<element name="X2" library="con-phoenix-508" package="MSTBA6" value="MSTBA6" x="25.638125" y="52.07" rot="R270">
+<attribute name="OC_NEWARK" value="71C4165" x="25.638125" y="52.07" size="1.778" layer="27" rot="R270" display="off"/>
+<attribute name="MPN" value="1757284" x="25.638125" y="52.07" size="1.778" layer="27" rot="R270" display="off"/>
+<attribute name="MF" value="FARNELL" x="25.638125" y="52.07" size="1.778" layer="27" rot="R270" display="off"/>
+<attribute name="OC_FARNELL" value="3705213" x="25.638125" y="52.07" size="1.778" layer="27" rot="R270" display="off"/>
 </element>
-<element name="J3" library="SparkFun-Connectors" package="USB-MICROB" value="USB-MICROB" x="25.161875" y="10.95375" rot="R270">
-<attribute name="PROD_ID" value="CONN-09505" x="25.161875" y="10.95375" size="1.778" layer="27" rot="R270" display="off"/>
+<element name="J3" library="SparkFun-Connectors" package="USB-MICROB" value="USB-MICROB" x="23.495" y="27.14625" rot="R270">
+<attribute name="PROD_ID" value="CONN-09505" x="23.495" y="27.14625" size="1.778" layer="27" rot="R270" display="off"/>
 </element>
-<element name="J4" library="SparkFun-Connectors" package="1X05_LOCK_LONGPADS" value="" x="112.7125" y="85.169375" rot="R180"/>
+<element name="J5" library="SparkFun-Connectors" package="MOLEX-1X6" value="" x="23.495" y="96.758125" rot="R270"/>
 </elements>
 <signals>
@@
 <contactref element="U3" pad="1"/>
 <contactref element="C11" pad="2"/>
+<contactref element="J5" pad="6"/>
+<wire x1="101.491875" y1="80.248125" x2="23.495" y2="84.058125" width="0" layer="19" extent="1-1"/>
+<wire x1="101.520625" y1="37.226875" x2="101.520625" y2="39.0525" width="0" layer="19" extent="1-1"/>
+<wire x1="87.2375" y1="67.355" x2="93.7375" y2="67.355" width="0" layer="19" extent="1-1"/>
 <wire x1="84.8175" y1="71.275" x2="87.2375" y2="67.355" width="0" layer="19" extent="1-1"/>
-<wire x1="93.7375" y1="67.355" x2="87.2375" y2="67.355" width="0" layer="19" extent="1-1"/>
-<wire x1="101.520625" y1="37.226875" x2="101.520625" y2="39.0525" width="0" layer="19" extent="1-1"/>
 <wire x1="90.17" y1="44.846875" x2="98.7425" y2="43.685" width="0" layer="19" extent="1-1"/>
 <wire x1="66.675" y1="40.35125" x2="70.6725" y2="37.62375" width="0" layer="19" extent="1-1"/>
@@
 <wire x1="68.659375" y1="17.4625" x2="68.29125" y2="21.034375" width="0" layer="19" extent="1-1"/>
 </signal>
-<signal name="N$6">
+<signal name="NRST">
 <contactref element="U2" pad="7"/>
 <contactref element="R3" pad="1"/>
@@
 <wire x1="79.295625" y1="74.215625" x2="78.819375" y2="73.739375" width="0.3048" layer="1"/>
 <wire x1="78.819375" y1="73.739375" x2="77.47" y2="73.739375" width="0.3048" layer="1"/>
+<contactref element="J5" pad="5"/>
+<wire x1="84.8175" y1="73.775" x2="23.495" y2="86.598125" width="0" layer="19" extent="1-1"/>
 </signal>
 <signal name="N$14">
@@
 <wire x1="96.1575" y1="78.03125" x2="98.374375" y2="80.248125" width="0.3048" layer="1"/>
 <contactref element="U3" pad="4"/>
-<wire x1="87.7375" y1="67.355" x2="94.2375" y2="67.355" width="0" layer="19" extent="1-1"/>
+<contactref element="J5" pad="2"/>
+<wire x1="98.374375" y1="80.248125" x2="23.495" y2="94.218125" width="0" layer="19" extent="1-1"/>
 <wire x1="86.7375" y1="78.695" x2="89.395625" y2="76.775" width="0" layer="19" extent="1-1"/>
 <wire x1="83.15625" y1="81.28" x2="85.4075" y2="79.21625" width="0" layer="19" extent="1-1"/>
+<wire x1="94.2375" y1="67.355" x2="87.7375" y2="67.355" width="0" layer="19" extent="1-1"/>
 <wire x1="66.754375" y1="66.119375" x2="79.136875" y2="70.723125" width="0" layer="19" extent="1-1"/>
 <wire x1="73.025" y1="55.40375" x2="66.754375" y2="66.119375" width="0" layer="19" extent="1-1"/>
@@
 <wire x1="71.199375" y1="17.4625" x2="71.40875" y2="21.034375" width="0" layer="19" extent="1-1"/>
 </signal>
+<signal name="N$11">
+<contactref element="J5" pad="1"/>
+<contactref element="U2" pad="55"/>
+<wire x1="91.2375" y1="78.695" x2="23.495" y2="96.758125" width="0" layer="19" extent="1-1"/>
+</signal>
+<signal name="SWDIO">
+<contactref element="U2" pad="46"/>
+<contactref element="J5" pad="3"/>
+<wire x1="96.1575" y1="75.775" x2="97.920625" y2="75.775" width="0.3048" layer="1"/>
+<wire x1="97.920625" y1="75.775" x2="98.821875" y2="76.67625" width="0.3048" layer="1"/>
+<wire x1="98.821875" y1="76.67625" x2="98.821875" y2="77.62875" width="0.3048" layer="1"/>
+<wire x1="98.821875" y1="77.62875" x2="99.139375" y2="77.94625" width="0.3048" layer="1"/>
+<wire x1="99.139375" y1="77.94625" x2="23.495" y2="91.678125" width="0" layer="19" extent="1-1"/>
+</signal>
+<signal name="SWCLK">
+<contactref element="U2" pad="49"/>
+<contactref element="J5" pad="4"/>
+<wire x1="94.2375" y1="78.695" x2="95.443125" y2="78.695" width="0.3048" layer="1"/>
+<wire x1="95.443125" y1="78.695" x2="96.67875" y2="79.930625" width="0.3048" layer="1"/>
+<wire x1="96.67875" y1="79.930625" x2="96.67875" y2="81.359375" width="0.3048" layer="1"/>
+<wire x1="96.67875" y1="81.359375" x2="97.393125" y2="82.07375" width="0.3048" layer="1"/>
+<wire x1="97.393125" y1="82.07375" x2="23.495" y2="89.138125" width="0" layer="19" extent="1-1"/>
+</signal>
 </signals>
