File: STM32F107RC.ETH.brd (EAGLE design)
At the start: 160 x 100 mm, 43 parts, among them J1 HR911105A, J3 USB-MICROB, Q1 8MHz, U1 LAN8720A-CP, U2 STM32F107RCT6, U3 LM1117MP-3.3, X1 CB3LV-3I-74M2500, X2 MSTBA6

Commit message: u 9-11-18
Parts:
- flipped J5 to the bottom
- flipped X2 to the bottom
Routing:
- net SWDIO: track 4.44 -> 102.4 mm, vias 0 -> 4
- net N$11: track 0.00 -> 81.8 mm, vias 0 -> 2
- net SWCLK: track 5.39 -> 80.2 mm, vias 0 -> 2

Commit message: u 10-11-18
Parts:
- removed J3: USB-MICROB, SparkFun-Connectors:USB-MICROB
- added J4: USB-MICROB", SparkFun-Connectors:USB-B-MICRO-SMD_V03
- moved J1 61.4 mm to (29.1, 12.9), turned to 270 degrees
Connections:
- net N$11 renamed SWO
- new net N$11: J4.D-, U2.44
- new net N$28: J4.D+, U2.45
- new net N$6: J4.VBUS, U2.42
- net GND: now also J4.GND
Routing:
- net LED1: track 35.9 -> 7.53 mm
- net LED2: track 35.7 -> 13.2 mm
- net GND: track 197.9 -> 187.0 mm
- net RD+: track 39.1 -> 31.1 mm
- net TD+: track 46.0 -> 41.3 mm
- net TD-: track 32.8 -> 29.2 mm
- net RD-: track 25.5 -> 23.2 mm
- net AVDD: track 56.9 -> 55.1 mm

Commit message: u 10-11-18 added USB OPTO INPUT;
Parts:
- added LED1, LED2, LED3: (no value), led:CHIPLED_0805
- added R19, R20, R21: (no value), SparkFun-Resistors:0805
- added U4: TLP281-4GB(F), TLP281-4GB_F_:SOIC127P700X210-16N
Connections:
- new net N$29: R19.1, X2.1
- new net N$30: R20.1, X2.2
- new net N$31: R21.1, X2.3
- new net N$32: LED1.C, R19.2
- new net N$33: LED2.C, R20.2
- new net N$34: LED3.C, R21.2
- new net N$35: LED1.A, U4.2
- new net N$36: LED2.A, U4.4
- new net N$37: LED3.A, U4.6
- new net N$38: U4.1, U4.3, U4.5
Changed lines of the file:
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@@
 <setting verticaltext="up"/>
 </settings>
-<grid distance="3.125" unitdist="mil" unit="mil" style="lines" multiple="1" display="yes" altdistance="0.025" altunitdist="inch" altunit="inch"/>
+<grid distance="6.26" unitdist="mil" unit="mil" style="lines" multiple="1" display="yes" altdistance="0.025" altunitdist="inch" altunit="inch"/>
 <layers>
 <layer number="1" name="Top" color="4" fill="1" visible="yes" active="yes"/>
@@
 <attribute name="PROD_ID" value="CONN-11752" x="20.47875" y="28.73375" size="1.778" layer="27" display="off"/>
 </element>
+<element name="U4" library="TLP281-4GB_F_" package="SOIC127P700X210-16N" value="TLP281-4GB(F)" x="57.4675" y="52.943125">
+<attribute name="PACKAGE" value="SOP-16 Toshiba" x="57.4675" y="52.943125" size="1.778" layer="27" display="off"/>
+<attribute name="AVAILABILITY" value="Unavailable" x="57.4675" y="52.943125" size="1.778" layer="27" display="off"/>
+<attribute name="MP" value="TLP281-4GB_F_" x="57.4675" y="52.943125" size="1.778" layer="27" display="off"/>
+<attribute name="PRICE" value="None" x="57.4675" y="52.943125" size="1.778" layer="27" display="off"/>
+<attribute name="DESCRIPTION" value=" Optocoupler DC-IN 4-CH Transistor DC-OUT 16-Pin SOP " x="57.4675" y="52.943125" size="1.778" layer="27" display="off"/>
+<attribute name="MF" value="Toshiba" x="57.4675" y="52.943125" size="1.778" layer="27" display="off"/>
+</element>
+<element name="LED1" library="led" package="CHIPLED_0805" value="" x="46.19625" y="56.118125" rot="R90"/>
+<element name="R19" library="SparkFun-Resistors" package="0805" value="" x="35.321875" y="64.77"/>
+<element name="R20" library="SparkFun-Resistors" package="0805" value="" x="35.251771875" y="59.62345"/>
+<element name="R21" library="SparkFun-Resistors" package="0805" value="" x="35.336225" y="54.694328125"/>
+<element name="LED2" library="led" package="CHIPLED_0805" value="" x="46.19625" y="53.578125" rot="R90"/>
+<element name="LED3" library="led" package="CHIPLED_0805" value="" x="46.19625" y="51.038125" rot="R90"/>
 </elements>
 <signals>
@@
 <wire x1="23.20375" y1="28.73375" x2="96.1575" y2="75.275" width="0" layer="19" extent="1-1"/>
 </signal>
+<signal name="N$29">
+<contactref element="X2" pad="1"/>
+<contactref element="R19" pad="1"/>
+<wire x1="34.421875" y1="64.77" x2="20.558125" y2="64.77" width="0" layer="19" extent="1-1"/>
+</signal>
+<signal name="N$30">
+<contactref element="X2" pad="2"/>
+<contactref element="R20" pad="1"/>
+<wire x1="34.351771875" y1="59.62345" x2="20.558125" y2="59.69" width="0" layer="19" extent="1-1"/>
+</signal>
+<signal name="N$31">
+<contactref element="R21" pad="1"/>
+<contactref element="X2" pad="3"/>
+<wire x1="34.436225" y1="54.694328125" x2="20.558125" y2="54.61" width="0" layer="19" extent="1-1"/>
+</signal>
+<signal name="N$32">
+<contactref element="R19" pad="2"/>
+<contactref element="LED1" pad="C"/>
+<wire x1="45.14625" y1="56.118125" x2="36.221875" y2="64.77" width="0" layer="19" extent="1-1"/>
+</signal>
+<signal name="N$33">
+<contactref element="LED2" pad="C"/>
+<contactref element="R20" pad="2"/>
+<wire x1="36.151771875" y1="59.62345" x2="45.14625" y2="53.578125" width="0" layer="19" extent="1-1"/>
+</signal>
+<signal name="N$34">
+<contactref element="R21" pad="2"/>
+<contactref element="LED3" pad="C"/>
+<wire x1="36.236225" y1="54.694328125" x2="45.14625" y2="51.038125" width="0" layer="19" extent="1-1"/>
+</signal>
+<signal name="N$35">
+<contactref element="LED1" pad="A"/>
+<contactref element="U4" pad="2"/>
+<wire x1="54.3125" y1="56.118125" x2="47.24625" y2="56.118125" width="0" layer="19" extent="1-1"/>
+</signal>
+<signal name="N$36">
+<contactref element="LED2" pad="A"/>
+<contactref element="U4" pad="4"/>
+<wire x1="54.3125" y1="53.578125" x2="47.24625" y2="53.578125" width="0" layer="19" extent="1-1"/>
+</signal>
+<signal name="N$37">
+<contactref element="LED3" pad="A"/>
+<contactref element="U4" pad="6"/>
+<wire x1="54.3125" y1="51.038125" x2="47.24625" y2="51.038125" width="0" layer="19" extent="1-1"/>
+</signal>
+<signal name="N$38">
+<contactref element="U4" pad="5"/>
+<contactref element="U4" pad="1"/>
+<contactref element="U4" pad="3"/>
+<wire x1="54.3125" y1="54.848125" x2="54.3125" y2="57.388125" width="0" layer="19" extent="1-1"/>
+<wire x1="54.3125" y1="52.308125" x2="54.3125" y2="54.848125" width="0" layer="19" extent="1-1"/>
+</signal>
 </signals>

Commit message: u 12-11-18
Parts:
- added LED4, LED5: (no value), led:CHIPLED_0805
- added R22, R23: (no value), SparkFun-Resistors:0805
- added U5: TLP281-4GB(F), TLP281-4GB_F_:SOIC127P700X210-16N
- added X3: MSTBA6, con-phoenix-508:MSTBA6
- moved J4 127.5 mm to (137.3, 80.0), turned to 180 degrees
- moved J5 68.2 mm to (91.7, 95.3), turned to 0 degrees
- moved LED1 9.82 mm to (41.4, 64.7)
- moved U4 9.61 mm to (49.0, 57.6)
- moved LED2 7.70 mm to (41.4, 59.6)
- moved LED3 6.01 mm to (41.4, 54.7)
Connections:
- new net N$39: R22.1, X2.4
- new net N$40: LED4.C, R22.2
- new net N$41: LED4.A, U4.8
- new net N$45: R23.1, X2.5
- new net N$46: LED5.C, R23.2
- new net N$47: LED5.A, U5.2
- net N$38: now also U4.7, U5.1, X2.6
Routing:
- net SWDIO: track 102.4 -> 21.9 mm, vias 4 -> 1
- net SWO: track 81.8 -> 11.3 mm, vias 2 -> 1
- net SWCLK: track 80.2 -> 11.8 mm, vias 2 -> 1
- net N$43: track 0.00 -> 32.1 mm
Other:
- board size 160 x 100 mm -> 160 x 114.6 mm

Commit message: omron relay library added. 12-11-18
Parts:
- added U$1: OMRON-RELAY-G5NB, omron-G5NB-1A-E:OMRON-G5NB
- moved X3 99.0 mm to (23.4, 88.7), turned to 270 degrees
- moved X2 3.24 mm to (22.5, 53.0), turned to 90 degrees
Changed lines of the file:
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@@
 <attribute name="SPICEPREFIX" value="C" x="69.85" y="21.034375" size="1.778" layer="27" rot="R180" display="off"/>
 </element>
-<element name="X2" library="con-phoenix-508" package="MSTBA6" value="MSTBA6" x="25.638125" y="52.07" rot="MR270">
-<attribute name="OC_NEWARK" value="71C4165" x="25.638125" y="52.07" size="1.778" layer="28" rot="MR270" display="off"/>
-<attribute name="MPN" value="1757284" x="25.638125" y="52.07" size="1.778" layer="28" rot="MR270" display="off"/>
-<attribute name="MF" value="FARNELL" x="25.638125" y="52.07" size="1.778" layer="28" rot="MR270" display="off"/>
-<attribute name="OC_FARNELL" value="3705213" x="25.638125" y="52.07" size="1.778" layer="28" rot="MR270" display="off"/>
+<element name="X2" library="con-phoenix-508" package="MSTBA6" value="MSTBA6" x="22.5400875" y="53.03164375" rot="MR90">
+<attribute name="OC_NEWARK" value="71C4165" x="22.5400875" y="53.03164375" size="1.778" layer="28" rot="MR90" display="off"/>
+<attribute name="MPN" value="1757284" x="22.5400875" y="53.03164375" size="1.778" layer="28" rot="MR90" display="off"/>
+<attribute name="MF" value="FARNELL" x="22.5400875" y="53.03164375" size="1.778" layer="28" rot="MR90" display="off"/>
+<attribute name="OC_FARNELL" value="3705213" x="22.5400875" y="53.03164375" size="1.778" layer="28" rot="MR90" display="off"/>
 </element>
 <element name="J5" library="SparkFun-Connectors" package="MOLEX-1X6" value="" x="91.669996875" y="95.2809875" rot="MR0"/>
@@
 <element name="R23" library="SparkFun-Resistors" package="0805" value="" x="35.2988875" y="44.52111875"/>
 <element name="LED5" library="led" package="CHIPLED_0805" value="" x="41.500046875" y="44.521121875" rot="R90"/>
-<element name="X3" library="con-phoenix-508" package="MSTBA6" value="MSTBA6" x="16.854425" y="-10.017253125">
-<attribute name="OC_NEWARK" value="71C4165" x="16.854425" y="-10.017253125" size="1.778" layer="27" display="off"/>
-<attribute name="MPN" value="1757284" x="16.854425" y="-10.017253125" size="1.778" layer="27" display="off"/>
-<attribute name="MF" value="FARNELL" x="16.854425" y="-10.017253125" size="1.778" layer="27" display="off"/>
-<attribute name="OC_FARNELL" value="3705213" x="16.854425" y="-10.017253125" size="1.778" layer="27" display="off"/>
+<element name="X3" library="con-phoenix-508" package="MSTBA6" value="MSTBA6" x="23.3735875" y="88.72423125" rot="R270">
+<attribute name="OC_NEWARK" value="71C4165" x="23.3735875" y="88.72423125" size="1.778" layer="27" rot="R270" display="off"/>
+<attribute name="MPN" value="1757284" x="23.3735875" y="88.72423125" size="1.778" layer="27" rot="R270" display="off"/>
+<attribute name="MF" value="FARNELL" x="23.3735875" y="88.72423125" size="1.778" layer="27" rot="R270" display="off"/>
+<attribute name="OC_FARNELL" value="3705213" x="23.3735875" y="88.72423125" size="1.778" layer="27" rot="R270" display="off"/>
 </element>
+<element name="U$1" library="omron-G5NB-1A-E" package="OMRON-G5NB" value="OMRON-RELAY-G5NB" x="133.08635" y="61.057534375"/>
 </elements>
 <signals>
@@
 <contactref element="X2" pad="1"/>
 <contactref element="R19" pad="1"/>
-<wire x1="20.558125" y1="64.77" x2="34.421875" y2="64.77" width="0" layer="19" extent="1-1"/>
+<wire x1="27.6200875" y1="40.33164375" x2="34.421875" y2="64.77" width="0" layer="19" extent="1-1"/>
 </signal>
 <signal name="N$30">
 <contactref element="X2" pad="2"/>
 <contactref element="R20" pad="1"/>
-<wire x1="20.558125" y1="59.69" x2="34.351771875" y2="59.62345" width="0" layer="19" extent="1-1"/>
+<wire x1="27.6200875" y1="45.41164375" x2="34.351771875" y2="59.62345" width="0" layer="19" extent="1-1"/>
 </signal>
 <signal name="N$31">
 <contactref element="R21" pad="1"/>
 <contactref element="X2" pad="3"/>
-<wire x1="20.558125" y1="54.61" x2="34.436225" y2="54.694328125" width="0" layer="19" extent="1-1"/>
+<wire x1="27.6200875" y1="50.49164375" x2="34.436225" y2="54.694328125" width="0" layer="19" extent="1-1"/>
 </signal>
 <signal name="N$32">
@@
 <wire x1="45.8852875" y1="54.379240625" x2="45.8852875" y2="56.919240625" width="0" layer="19" extent="1-1"/>
 <wire x1="45.977234375" y1="45.786040625" x2="45.8852875" y2="54.379240625" width="0" layer="19" extent="1-1"/>
-<wire x1="20.558125" y1="39.37" x2="45.977234375" y2="45.786040625" width="0" layer="19" extent="1-1"/>
+<wire x1="27.6200875" y1="65.73164375" x2="45.977234375" y2="45.786040625" width="0" layer="19" extent="1-1"/>
 </signal>
 <signal name="N$39">
 <contactref element="X2" pad="4"/>
 <contactref element="R22" pad="1"/>
-<wire x1="20.558125" y1="49.53" x2="34.3988875" y2="49.609246875" width="0" layer="19" extent="1-1"/>
+<wire x1="27.6200875" y1="55.57164375" x2="34.3988875" y2="49.609246875" width="0" layer="19" extent="1-1"/>
 </signal>
 <signal name="N$40">
@@
 <contactref element="X2" pad="5"/>
 <contactref element="R23" pad="1"/>
-<wire x1="20.558125" y1="44.45" x2="34.3988875" y2="44.52111875" width="0" layer="19" extent="1-1"/>
+<wire x1="27.6200875" y1="60.65164375" x2="34.3988875" y2="44.52111875" width="0" layer="19" extent="1-1"/>
 </signal>
 <signal name="N$46">

Commit message: u 11/28/18
Parts:
- moved X3 1.28 mm to (22.1, 88.6)
- moved X2 1.07 mm to (22.1, 52.1), flipped to the top, turned to 270 degrees
Routing:
- net N$42: track 0.00 -> 9.70 mm
Changed lines of the file:
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@@
 <attribute name="SPICEPREFIX" value="C" x="69.85" y="21.034375" size="1.778" layer="27" rot="R180" display="off"/>
 </element>
-<element name="X2" library="con-phoenix-508" package="MSTBA6" value="MSTBA6" x="22.5400875" y="53.03164375" rot="MR90">
-<attribute name="OC_NEWARK" value="71C4165" x="22.5400875" y="53.03164375" size="1.778" layer="28" rot="MR90" display="off"/>
-<attribute name="MPN" value="1757284" x="22.5400875" y="53.03164375" size="1.778" layer="28" rot="MR90" display="off"/>
-<attribute name="MF" value="FARNELL" x="22.5400875" y="53.03164375" size="1.778" layer="28" rot="MR90" display="off"/>
-<attribute name="OC_FARNELL" value="3705213" x="22.5400875" y="53.03164375" size="1.778" layer="28" rot="MR90" display="off"/>
+<element name="X2" library="con-phoenix-508" package="MSTBA6" value="MSTBA6" x="22.063075" y="52.069996875" rot="R270">
+<attribute name="OC_NEWARK" value="71C4165" x="22.063075" y="52.069996875" size="1.778" layer="27" rot="R270" display="off"/>
+<attribute name="MPN" value="1757284" x="22.063075" y="52.069996875" size="1.778" layer="27" rot="R270" display="off"/>
+<attribute name="MF" value="FARNELL" x="22.063075" y="52.069996875" size="1.778" layer="27" rot="R270" display="off"/>
+<attribute name="OC_FARNELL" value="3705213" x="22.063075" y="52.069996875" size="1.778" layer="27" rot="R270" display="off"/>
 </element>
 <element name="J5" library="SparkFun-Connectors" package="MOLEX-1X6" value="" x="91.669996875" y="95.2809875" rot="MR0"/>
@@
 <element name="R23" library="SparkFun-Resistors" package="0805" value="" x="35.2988875" y="44.52111875"/>
 <element name="LED5" library="led" package="CHIPLED_0805" value="" x="41.500046875" y="44.521121875" rot="R90"/>
-<element name="X3" library="con-phoenix-508" package="MSTBA6" value="MSTBA6" x="23.3735875" y="88.72423125" rot="R270">
-<attribute name="OC_NEWARK" value="71C4165" x="23.3735875" y="88.72423125" size="1.778" layer="27" rot="R270" display="off"/>
-<attribute name="MPN" value="1757284" x="23.3735875" y="88.72423125" size="1.778" layer="27" rot="R270" display="off"/>
-<attribute name="MF" value="FARNELL" x="23.3735875" y="88.72423125" size="1.778" layer="27" rot="R270" display="off"/>
-<attribute name="OC_FARNELL" value="3705213" x="23.3735875" y="88.72423125" size="1.778" layer="27" rot="R270" display="off"/>
+<element name="X3" library="con-phoenix-508" package="MSTBA6" value="MSTBA6" x="22.10155625" y="88.565228125" rot="R270">
+<attribute name="OC_NEWARK" value="71C4165" x="22.10155625" y="88.565228125" size="1.778" layer="27" rot="R270" display="off"/>
+<attribute name="MPN" value="1757284" x="22.10155625" y="88.565228125" size="1.778" layer="27" rot="R270" display="off"/>
+<attribute name="MF" value="FARNELL" x="22.10155625" y="88.565228125" size="1.778" layer="27" rot="R270" display="off"/>
+<attribute name="OC_FARNELL" value="3705213" x="22.10155625" y="88.565228125" size="1.778" layer="27" rot="R270" display="off"/>
 </element>
 <element name="U$1" library="omron-G5NB-1A-E" package="OMRON-G5NB" value="OMRON-RELAY-G5NB" x="133.08635" y="61.057534375"/>
@@
 <contactref element="X2" pad="1"/>
 <contactref element="R19" pad="1"/>
-<wire x1="27.6200875" y1="40.33164375" x2="34.421875" y2="64.77" width="0" layer="19" extent="1-1"/>
+<wire x1="27.143075" y1="64.769996875" x2="34.421875" y2="64.77" width="0" layer="19" extent="1-1"/>
 </signal>
 <signal name="N$30">
 <contactref element="X2" pad="2"/>
 <contactref element="R20" pad="1"/>
-<wire x1="27.6200875" y1="45.41164375" x2="34.351771875" y2="59.62345" width="0" layer="19" extent="1-1"/>
+<wire x1="27.143075" y1="59.689996875" x2="34.351771875" y2="59.62345" width="0" layer="19" extent="1-1"/>
 </signal>
 <signal name="N$31">
 <contactref element="R21" pad="1"/>
 <contactref element="X2" pad="3"/>
-<wire x1="27.6200875" y1="50.49164375" x2="34.436225" y2="54.694328125" width="0" layer="19" extent="1-1"/>
+<wire x1="27.143075" y1="54.609996875" x2="34.436225" y2="54.694328125" width="0" layer="19" extent="1-1"/>
 </signal>
 <signal name="N$32">
@@
 <wire x1="45.8852875" y1="54.379240625" x2="45.8852875" y2="56.919240625" width="0" layer="19" extent="1-1"/>
 <wire x1="45.977234375" y1="45.786040625" x2="45.8852875" y2="54.379240625" width="0" layer="19" extent="1-1"/>
-<wire x1="27.6200875" y1="65.73164375" x2="45.977234375" y2="45.786040625" width="0" layer="19" extent="1-1"/>
+<wire x1="27.143075" y1="39.369996875" x2="45.977234375" y2="45.786040625" width="0" layer="19" extent="1-1"/>
 </signal>
 <signal name="N$39">
 <contactref element="X2" pad="4"/>
 <contactref element="R22" pad="1"/>
-<wire x1="27.6200875" y1="55.57164375" x2="34.3988875" y2="49.609246875" width="0" layer="19" extent="1-1"/>
+<wire x1="27.143075" y1="49.529996875" x2="34.3988875" y2="49.609246875" width="0" layer="19" extent="1-1"/>
 </signal>
 <signal name="N$40">
@@
 <contactref element="X2" pad="5"/>
 <contactref element="R23" pad="1"/>
-<wire x1="27.6200875" y1="60.65164375" x2="34.3988875" y2="44.52111875" width="0" layer="19" extent="1-1"/>
+<wire x1="27.143075" y1="44.449996875" x2="34.3988875" y2="44.52111875" width="0" layer="19" extent="1-1"/>
 </signal>
 <signal name="N$46">
@@
 <wire x1="42.550046875" y1="44.521121875" x2="45.977234375" y2="44.516040625" width="0" layer="19" extent="1-1"/>
 </signal>
+<signal name="N$42">
+<wire x1="17.17243125" y1="67.417696875" x2="17.17243125" y2="77.116940625" width="0.254" layer="16"/>
+</signal>
 </signals>

Commit message: U01.12.18
Parts:
- added IC1: LM358, SparkFun-AnalogIC:DIP08
Connections:
- new net V+: IC1.8
- new net V-: IC1.4
Changed lines of the file:
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@@
 </element>
 <element name="U$1" library="omron-G5NB-1A-E" package="OMRON-G5NB" value="OMRON-RELAY-G5NB" x="133.08635" y="61.057534375"/>
+<element name="IC1" library="SparkFun-AnalogIC" package="DIP08" value="LM358" x="7.4731875" y="-4.929125">
+<attribute name="PROD_ID" value="IC-09172" x="7.4731875" y="-4.929125" size="1.778" layer="27" display="off"/>
+</element>
 </elements>
 <signals>
@@
 <wire x1="17.17243125" y1="67.417696875" x2="17.17243125" y2="77.116940625" width="0.254" layer="16"/>
 </signal>
+<signal name="V+">
+<contactref element="IC1" pad="8"/>
+</signal>
+<signal name="V-">
+<contactref element="IC1" pad="4"/>
+</signal>
 </signals>

Commit message: uu
Parts:
- removed IC1: LM358, SparkFun-AnalogIC:DIP08
- added C12, C14: 0.1uF, SparkFun-Capacitors:0603-CAP
- added IC2: LM358, SparkFun-AnalogIC:LM358_DIP08
- added R24, R30: 0.3, SparkFun-Resistors:0805
- added R25, R26, R27, R28, R29, R32, R33, R34, R35, R36: 1K, SparkFun-Resistors:AXIAL-0.3
- added SJ1, SJ2: (no value), jumper:SJ_2
Connections:
- removed net V-: IC1.4
- new net N$44: C12.2, IC2.6, R25.P$1, R26.P$2, R29.P$1
- new net N$48: IC2.5, R27.P$2, R28.P$1
- new net N$49: IC2.7, R25.P$2, R30.1
- new net N$50: R28.P$2, SJ2.1
- new net N$51: R29.P$2, SJ2.3
- new net N$55: IC2.2, R32.P$1, R34.P$2, R35.P$1
- new net N$56: C14.2, IC2.3, R33.P$2, R36.P$1
- new net N$58: IC2.1, R24.1, R32.P$2
- new net N$60: R35.P$2, SJ1.1
- new net N$61: R36.P$2, SJ1.3
- net GND: now also C12.1, C14.1, IC2.4, R26.P$1, R27.P$1, R33.P$1, R34.P$1
- net V+: now also IC2.8; no longer IC1.8
Routing:
- net N$56: track 0.00 -> 18.3 mm
- net N$55: track 0.00 -> 15.9 mm, vias 0 -> 2
- net N$58: track 0.00 -> 8.18 mm
