File: STM32F107RC.ETH.sch (EAGLE design)
At the start: 28 parts, among them J1 HR911105A, Q1 8MHz, U1 LAN8720A-CP, U2 STM32F107RCT6, X1 CB3LV-3I-74M2500

Commit message: Add files via upload
Parts:
- J2: device SparkFun-Connectors:M01SMD -> SparkFun-Connectors:M01OFFSET
Connections:
- new net LED1: J1.GC, U1.LED1/REGOFF
- new net LED2: J1.YC, U1.LED2/!NINTSEL!
- new net N$23: J1.TD+, U1.TXP
- new net N$28: J1.TD-, U1.TXN
- new net N$29: J1.RD+, U1.RXP
- new net N$31: J1.RD-, U1.RXN
- net VCC: now also J1.GA, J1.P4, J1.P5, J1.YA, JP1.3
Other:
- moved on the sheet: J2
Changed lines of the file:
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@@
 <parts>
 <part name="U1" library="LAN8720A-CP" deviceset="LAN8720A-CP" device=""/>
-<part name="J2" library="SparkFun-Connectors" deviceset="M01" device="SMD"/>
 <part name="R1" library="resistor" deviceset="R-EU_" device="0204_7" value="1K5"/>
 <part name="R2" library="resistor" deviceset="R-EU_" device="0204_7" value="10"/>
@@
 <part name="C7" library="resistor" deviceset="C-EU" device="C1206" value="10uF"/>
 <part name="J1" library="HR911105A" deviceset="HR911105A" device=""/>
+<part name="J2" library="SparkFun-Connectors" deviceset="M01" device="OFFSET"/>
 </parts>
 <sheets>
@@
 <instances>
 <instance part="U1" gate="G$1" x="-25.4" y="154.94"/>
-<instance part="J2" gate="G$1" x="17.78" y="193.04" rot="R270"/>
 <instance part="R1" gate="G$1" x="12.7" y="182.88" rot="R90"/>
 <instance part="R2" gate="G$1" x="7.62" y="182.88" rot="R90"/>
@@
 <instance part="C7" gate="G$1" x="-51.7525" y="196.215" rot="R270"/>
 <instance part="J1" gate="G$1" x="-158.115" y="139.3825" rot="R180"/>
+<instance part="J2" gate="G$1" x="17.78" y="198.12" rot="R270"/>
 </instances>
 <busses>
@@
 <net name="N$10" class="0">
 <segment>
-<pinref part="J2" gate="G$1" pin="1"/>
 <wire x1="25.4" y1="91.44" x2="25.4" y2="185.42" width="0.1524" layer="91"/>
 <wire x1="25.4" y1="185.42" x2="17.78" y2="185.42" width="0.1524" layer="91"/>
 <pinref part="U2" gate="A" pin="PA8"/>
 <wire x1="81.28" y1="91.44" x2="25.4" y2="91.44" width="0.1524" layer="91"/>
+<pinref part="J2" gate="G$1" pin="1"/>
+<wire x1="17.78" y1="190.5" x2="17.145" y2="189.865" width="0.1524" layer="91"/>
+<wire x1="17.145" y1="189.865" x2="17.145" y2="186.055" width="0.1524" layer="91"/>
+<wire x1="17.145" y1="186.055" x2="17.78" y2="185.42" width="0.1524" layer="91"/>
 </segment>
 </net>
@@
 <pinref part="SUPPLY2" gate="G$1" pin="VCC"/>
 <wire x1="53.975" y1="141.2875" x2="53.975" y2="139.3825" width="0.1524" layer="91"/>
-<wire x1="74.93" y1="141.9225" x2="77.7875" y2="141.9225" width="0.1524" layer="91"/>
 <wire x1="77.7875" y1="141.9225" x2="78.74" y2="142.875" width="0.1524" layer="91"/>
 <wire x1="78.74" y1="142.875" x2="78.74" y2="145.415" width="0.1524" layer="91"/>
@@
 <wire x1="63.5" y1="142.5575" x2="62.23" y2="141.2875" width="0.1524" layer="91"/>
 <wire x1="62.23" y1="141.2875" x2="53.975" y2="141.2875" width="0.1524" layer="91"/>
+<pinref part="JP1" gate="1" pin="3"/>
+<wire x1="74.6125" y1="141.9225" x2="77.7875" y2="141.9225" width="0.1524" layer="91"/>
 </segment>
 <segment>
@@
 <wire x1="-99.695" y1="168.5925" x2="-96.2025" y2="172.085" width="0.1524" layer="91"/>
 <wire x1="-96.2025" y1="172.085" x2="-86.0425" y2="172.085" width="0.1524" layer="91"/>
+<pinref part="J1" gate="G$1" pin="P4"/>
+<wire x1="-120.015" y1="126.6825" x2="-113.665" y2="126.6825" width="0.1524" layer="91"/>
+<wire x1="-113.665" y1="126.6825" x2="-111.125" y2="129.2225" width="0.1524" layer="91"/>
+<wire x1="-111.125" y1="129.2225" x2="-111.125" y2="150.8125" width="0.1524" layer="91"/>
+<wire x1="-111.125" y1="150.8125" x2="-111.125" y2="163.195" width="0.1524" layer="91"/>
+<wire x1="-111.125" y1="163.195" x2="-111.125" y2="169.545" width="0.1524" layer="91"/>
+<wire x1="-111.125" y1="169.545" x2="-108.585" y2="172.085" width="0.1524" layer="91"/>
+<wire x1="-108.585" y1="172.085" x2="-105.7275" y2="172.085" width="0.1524" layer="91"/>
+<pinref part="J1" gate="G$1" pin="P5"/>
+<wire x1="-105.7275" y1="172.085" x2="-96.2025" y2="172.085" width="0.1524" layer="91"/>
+<wire x1="-120.015" y1="113.9825" x2="-106.9975" y2="113.9825" width="0.1524" layer="91"/>
+<wire x1="-106.9975" y1="113.9825" x2="-104.14" y2="116.84" width="0.1524" layer="91"/>
+<wire x1="-104.14" y1="116.84" x2="-104.14" y2="137.4775" width="0.1524" layer="91"/>
+<wire x1="-104.14" y1="137.4775" x2="-106.68" y2="140.0175" width="0.1524" layer="91"/>
+<wire x1="-106.68" y1="140.0175" x2="-106.68" y2="171.1325" width="0.1524" layer="91"/>
+<wire x1="-106.68" y1="171.1325" x2="-105.7275" y2="172.085" width="0.1524" layer="91"/>
+<pinref part="J1" gate="G$1" pin="GA"/>
+<wire x1="-120.015" y1="149.5425" x2="-112.395" y2="149.5425" width="0.1524" layer="91"/>
+<wire x1="-112.395" y1="149.5425" x2="-111.125" y2="150.8125" width="0.1524" layer="91"/>
+<pinref part="J1" gate="G$1" pin="YA"/>
+<wire x1="-120.015" y1="162.2425" x2="-112.0775" y2="162.2425" width="0.1524" layer="91"/>
+<wire x1="-112.0775" y1="162.2425" x2="-111.125" y2="163.195" width="0.1524" layer="91"/>
 </segment>
 </net>
@@
 </segment>
 </net>
+<net name="N$23" class="0">
+<segment>
+<pinref part="U1" gate="G$1" pin="TXP"/>
+<wire x1="-48.26" y1="144.78" x2="-50.4825" y2="144.78" width="0.1524" layer="91"/>
+<wire x1="-50.4825" y1="144.78" x2="-52.07" y2="143.1925" width="0.1524" layer="91"/>
+<wire x1="-52.07" y1="143.1925" x2="-80.9625" y2="143.1925" width="0.1524" layer="91"/>
+<wire x1="-80.9625" y1="143.1925" x2="-88.265" y2="135.89" width="0.1524" layer="91"/>
+<wire x1="-88.265" y1="135.89" x2="-113.3475" y2="135.89" width="0.1524" layer="91"/>
+<wire x1="-113.3475" y1="135.89" x2="-117.475" y2="131.7625" width="0.1524" layer="91"/>
+<pinref part="J1" gate="G$1" pin="TD+"/>
+<wire x1="-117.475" y1="131.7625" x2="-120.015" y2="131.7625" width="0.1524" layer="91"/>
+</segment>
+</net>
+<net name="N$28" class="0">
+<segment>
+<pinref part="U1" gate="G$1" pin="TXN"/>
+<wire x1="-48.26" y1="142.24" x2="-50.8" y2="142.24" width="0.1524" layer="91"/>
+<wire x1="-50.8" y1="142.24" x2="-52.07" y2="140.97" width="0.1524" layer="91"/>
+<wire x1="-52.07" y1="140.97" x2="-80.3275" y2="140.97" width="0.1524" layer="91"/>
+<wire x1="-80.3275" y1="140.97" x2="-96.2025" y2="125.095" width="0.1524" layer="91"/>
+<wire x1="-96.2025" y1="125.095" x2="-106.9975" y2="125.095" width="0.1524" layer="91"/>
+<pinref part="J1" gate="G$1" pin="TD-"/>
+<wire x1="-106.9975" y1="125.095" x2="-110.49" y2="121.6025" width="0.1524" layer="91"/>
+<wire x1="-110.49" y1="121.6025" x2="-120.015" y2="121.6025" width="0.1524" layer="91"/>
+</segment>
+</net>
+<net name="N$29" class="0">
+<segment>
+<pinref part="U1" gate="G$1" pin="RXP"/>
+<wire x1="-48.26" y1="139.7" x2="-51.1175" y2="139.7" width="0.1524" layer="91"/>
+<wire x1="-51.1175" y1="139.7" x2="-52.07" y2="138.7475" width="0.1524" layer="91"/>
+<wire x1="-52.07" y1="138.7475" x2="-77.47" y2="138.7475" width="0.1524" layer="91"/>
+<wire x1="-77.47" y1="138.7475" x2="-97.4725" y2="119.0625" width="0.1524" layer="91"/>
+<wire x1="-97.4725" y1="119.0625" x2="-105.41" y2="119.0625" width="0.1524" layer="91"/>
+<pinref part="J1" gate="G$1" pin="RD+"/>
+<wire x1="-105.41" y1="119.0625" x2="-120.015" y2="119.0625" width="0.1524" layer="91"/>
+</segment>
+</net>
+<net name="N$31" class="0">
+<segment>
+<pinref part="U1" gate="G$1" pin="RXN"/>
+<wire x1="-48.26" y1="137.16" x2="-51.1175" y2="137.16" width="0.1524" layer="91"/>
+<wire x1="-51.1175" y1="137.16" x2="-52.07" y2="136.2075" width="0.1524" layer="91"/>
+<wire x1="-52.07" y1="136.2075" x2="-76.5175" y2="136.2075" width="0.1524" layer="91"/>
+<wire x1="-76.5175" y1="136.2075" x2="-103.8225" y2="108.9025" width="0.1524" layer="91"/>
+<pinref part="J1" gate="G$1" pin="RD-"/>
+<wire x1="-103.8225" y1="108.9025" x2="-120.015" y2="108.9025" width="0.1524" layer="91"/>
+</segment>
+</net>
+<net name="LED2" class="0">
+<segment>
+<pinref part="U1" gate="G$1" pin="LED2/!NINTSEL!"/>
+<wire x1="-2.54" y1="142.24" x2="-1.905" y2="142.24" width="0.1524" layer="91"/>
+<wire x1="-1.905" y1="142.24" x2="-0.9525" y2="141.2875" width="0.1524" layer="91"/>
+<wire x1="-0.9525" y1="141.2875" x2="-0.9525" y2="126.365" width="0.1524" layer="91"/>
+<wire x1="-0.9525" y1="126.365" x2="-2.8575" y2="124.46" width="0.1524" layer="91"/>
+<wire x1="-2.8575" y1="124.46" x2="-31.115" y2="124.46" width="0.1524" layer="91"/>
+<wire x1="-31.115" y1="124.46" x2="-32.0675" y2="123.5075" width="0.1524" layer="91"/>
+<wire x1="-32.0675" y1="123.5075" x2="-43.18" y2="123.5075" width="0.1524" layer="91"/>
+<label x="-41.91" y="121.285" size="1.778" layer="95"/>
+</segment>
+<segment>
+<pinref part="J1" gate="G$1" pin="YC"/>
+<wire x1="-120.015" y1="167.3225" x2="-119.0625" y2="167.3225" width="0.1524" layer="91"/>
+<wire x1="-119.0625" y1="167.3225" x2="-117.7925" y2="168.5925" width="0.1524" layer="91"/>
+<wire x1="-117.7925" y1="168.5925" x2="-117.7925" y2="187.96" width="0.1524" layer="91"/>
+<label x="-118.4275" y="180.975" size="1.778" layer="95" rot="R90"/>
+</segment>
+</net>
+<net name="LED1" class="0">
+<segment>
+<pinref part="U1" gate="G$1" pin="LED1/REGOFF"/>
+<wire x1="-2.54" y1="144.78" x2="0.635" y2="144.78" width="0.1524" layer="91"/>
+<wire x1="0.635" y1="144.78" x2="1.5875" y2="143.8275" width="0.1524" layer="91"/>
+<wire x1="1.5875" y1="143.8275" x2="1.5875" y2="125.095" width="0.1524" layer="91"/>
+<wire x1="1.5875" y1="125.095" x2="-0.9525" y2="122.555" width="0.1524" layer="91"/>
+<wire x1="-0.9525" y1="122.555" x2="-22.225" y2="122.555" width="0.1524" layer="91"/>
+<wire x1="-22.225" y1="122.555" x2="-23.1775" y2="121.6025" width="0.1524" layer="91"/>
+<wire x1="-23.1775" y1="121.6025" x2="-33.655" y2="121.6025" width="0.1524" layer="91"/>
+<label x="-31.4325" y="119.38" size="1.778" layer="95"/>
+</segment>
+<segment>
+<pinref part="J1" gate="G$1" pin="GC"/>
+<wire x1="-120.015" y1="154.6225" x2="-115.8875" y2="154.6225" width="0.1524" layer="91"/>
+<wire x1="-115.8875" y1="154.6225" x2="-113.9825" y2="156.5275" width="0.1524" layer="91"/>
+<wire x1="-113.9825" y1="156.5275" x2="-113.9825" y2="169.545" width="0.1524" layer="91"/>
+<wire x1="-113.9825" y1="169.545" x2="-112.395" y2="171.1325" width="0.1524" layer="91"/>
+<wire x1="-112.395" y1="171.1325" x2="-112.395" y2="188.2775" width="0.1524" layer="91"/>
+<label x="-112.7125" y="181.2925" size="1.778" layer="95" rot="R90"/>
+</segment>
+</net>

Commit message: Add files via upload
Parts:
- added R13, R14: 330R, resistor:R-EU_0204_7
Connections:
- new net SIG_LED01: R14.2, U1.LED1/REGOFF
- new net SIG_LED02: R13.2, U1.LED2/!NINTSEL!
- net LED1: now also R14.1; no longer U1.LED1/REGOFF
- net LED2: now also R13.1; no longer U1.LED2/!NINTSEL!
- net N$4: now also U2.PA7
Changed lines of the file:
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@@
 <part name="J1" library="HR911105A" deviceset="HR911105A" device=""/>
 <part name="J2" library="SparkFun-Connectors" deviceset="M01" device="OFFSET"/>
+<part name="R13" library="resistor" deviceset="R-EU_" device="0204_7" value="330R"/>
+<part name="R14" library="resistor" deviceset="R-EU_" device="0204_7" value="330R"/>
 </parts>
 <sheets>
@@
 <instance part="J1" gate="G$1" x="-158.115" y="139.3825" rot="R180"/>
 <instance part="J2" gate="G$1" x="17.78" y="198.12" rot="R270"/>
+<instance part="R13" gate="G$1" x="-12.3825" y="124.46"/>
+<instance part="R14" gate="G$1" x="-12.3825" y="117.475"/>
 </instances>
 <busses>
@@
 <net name="N$4" class="0">
 <segment>
-<wire x1="81.5975" y1="93.98" x2="24.13" y2="93.98" width="0.1524" layer="91"/>
+<wire x1="81.28" y1="93.98" x2="24.13" y2="93.98" width="0.1524" layer="91"/>
 <pinref part="R9" gate="G$1" pin="2"/>
 <wire x1="22.86" y1="130.4925" x2="22.86" y2="95.25" width="0.1524" layer="91"/>
 <wire x1="22.86" y1="95.25" x2="24.13" y2="93.98" width="0.1524" layer="91"/>
+<pinref part="U2" gate="A" pin="PA7"/>
 </segment>
 </net>
@@
 <net name="LED2" class="0">
 <segment>
-<pinref part="U1" gate="G$1" pin="LED2/!NINTSEL!"/>
-<wire x1="-2.54" y1="142.24" x2="-1.905" y2="142.24" width="0.1524" layer="91"/>
-<wire x1="-1.905" y1="142.24" x2="-0.9525" y2="141.2875" width="0.1524" layer="91"/>
-<wire x1="-0.9525" y1="141.2875" x2="-0.9525" y2="126.365" width="0.1524" layer="91"/>
-<wire x1="-0.9525" y1="126.365" x2="-2.8575" y2="124.46" width="0.1524" layer="91"/>
-<wire x1="-2.8575" y1="124.46" x2="-31.115" y2="124.46" width="0.1524" layer="91"/>
-<wire x1="-31.115" y1="124.46" x2="-32.0675" y2="123.5075" width="0.1524" layer="91"/>
-<wire x1="-32.0675" y1="123.5075" x2="-43.18" y2="123.5075" width="0.1524" layer="91"/>
-<label x="-41.91" y="121.285" size="1.778" layer="95"/>
-</segment>
-<segment>
 <pinref part="J1" gate="G$1" pin="YC"/>
 <wire x1="-120.015" y1="167.3225" x2="-119.0625" y2="167.3225" width="0.1524" layer="91"/>
@@
 <label x="-118.4275" y="180.975" size="1.778" layer="95" rot="R90"/>
 </segment>
+<segment>
+<pinref part="R13" gate="G$1" pin="1"/>
+<wire x1="-17.4625" y1="124.46" x2="-24.765" y2="124.46" width="0.1524" layer="91"/>
+<label x="-23.8125" y="125.095" size="1.778" layer="95"/>
+</segment>
 </net>
 <net name="LED1" class="0">
-<segment>
-<pinref part="U1" gate="G$1" pin="LED1/REGOFF"/>
-<wire x1="-2.54" y1="144.78" x2="0.635" y2="144.78" width="0.1524" layer="91"/>
-<wire x1="0.635" y1="144.78" x2="1.5875" y2="143.8275" width="0.1524" layer="91"/>
-<wire x1="1.5875" y1="143.8275" x2="1.5875" y2="125.095" width="0.1524" layer="91"/>
-<wire x1="1.5875" y1="125.095" x2="-0.9525" y2="122.555" width="0.1524" layer="91"/>
-<wire x1="-0.9525" y1="122.555" x2="-22.225" y2="122.555" width="0.1524" layer="91"/>
-<wire x1="-22.225" y1="122.555" x2="-23.1775" y2="121.6025" width="0.1524" layer="91"/>
-<wire x1="-23.1775" y1="121.6025" x2="-33.655" y2="121.6025" width="0.1524" layer="91"/>
-<label x="-31.4325" y="119.38" size="1.778" layer="95"/>
-</segment>
 <segment>
 <pinref part="J1" gate="G$1" pin="GC"/>
@@
 <label x="-112.7125" y="181.2925" size="1.778" layer="95" rot="R90"/>
 </segment>
-</net>
+<segment>
+<pinref part="R14" gate="G$1" pin="1"/>
+<wire x1="-17.4625" y1="117.475" x2="-30.7975" y2="117.475" width="0.1524" layer="91"/>
+<label x="-23.8125" y="117.7925" size="1.778" layer="95"/>
+</segment>
+</net>
+<net name="SIG_LED02" class="0">
+<segment>
+<pinref part="U1" gate="G$1" pin="LED2/!NINTSEL!"/>
+<wire x1="-2.54" y1="142.24" x2="-1.905" y2="142.24" width="0.1524" layer="91"/>
+<wire x1="-1.905" y1="142.24" x2="-0.9525" y2="141.2875" width="0.1524" layer="91"/>
+<wire x1="-0.9525" y1="141.2875" x2="-0.9525" y2="126.365" width="0.1524" layer="91"/>
+<wire x1="-0.9525" y1="126.365" x2="-2.8575" y2="124.46" width="0.1524" layer="91"/>
+<pinref part="R13" gate="G$1" pin="2"/>
+<wire x1="-2.8575" y1="124.46" x2="-7.3025" y2="124.46" width="0.1524" layer="91"/>
+</segment>
+</net>
+<net name="SIG_LED01" class="0">
+<segment>
+<pinref part="U1" gate="G$1" pin="LED1/REGOFF"/>
+<wire x1="-2.54" y1="144.78" x2="0.635" y2="144.78" width="0.1524" layer="91"/>
+<wire x1="0.635" y1="144.78" x2="1.5875" y2="143.8275" width="0.1524" layer="91"/>
+<wire x1="1.5875" y1="143.8275" x2="1.5875" y2="120.015" width="0.1524" layer="91"/>
+<wire x1="1.5875" y1="120.015" x2="-0.9525" y2="117.475" width="0.1524" layer="91"/>
+<pinref part="R14" gate="G$1" pin="2"/>
+<wire x1="-0.9525" y1="117.475" x2="-7.3025" y2="117.475" width="0.1524" layer="91"/>
+</segment>
+</net>

Commit message: Add files via upload
Parts:
- R5: value 12.1K -> 4K7
Connections:
- removed net N$11: L1.1, U1.VDD1A, U1.VDD2A
- new net AVDD: J1.P4, J1.P5, L1.1, U1.VDD1A, U1.VDD2A
- net VCC: no longer J1.P4, J1.P5
Changed lines of the file:
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@@
 <part name="SUPPLY2" library="supply2" deviceset="VCC" device=""/>
 <part name="R4" library="resistor" deviceset="R-EU_" device="0204_7" value="12.1K"/>
-<part name="R5" library="resistor" deviceset="R-EU_" device="0204_7" value="12.1K"/>
+<part name="R5" library="resistor" deviceset="R-EU_" device="0204_7" value="4K7"/>
 <part name="C4" library="resistor" deviceset="C-EU" device="C1206"/>
 <part name="SUPPLY7" library="supply2" deviceset="VCC" device=""/>
@@
 </segment>
 </net>
-<net name="N$11" class="0">
+<net name="AVDD" class="0">
 <segment>
 <pinref part="U1" gate="G$1" pin="VDD1A"/>
@@
 <pinref part="L1" gate="G$1" pin="1"/>
 <junction x="0" y="195.58"/>
+<label x="-9.8425" y="196.5325" size="1.778" layer="95"/>
+<wire x1="-113.665" y1="126.6825" x2="-111.125" y2="129.2225" width="0.1524" layer="91"/>
+<pinref part="J1" gate="G$1" pin="P4"/>
+<wire x1="-120.015" y1="126.6825" x2="-113.665" y2="126.6825" width="0.1524" layer="91"/>
+<wire x1="-111.125" y1="129.2225" x2="-111.125" y2="137.4775" width="0.1524" layer="91"/>
+<wire x1="-111.125" y1="137.4775" x2="-108.585" y2="140.0175" width="0.1524" layer="91"/>
+<wire x1="-104.14" y1="137.4775" x2="-106.68" y2="140.0175" width="0.1524" layer="91"/>
+<wire x1="-104.14" y1="116.84" x2="-104.14" y2="137.4775" width="0.1524" layer="91"/>
+<pinref part="J1" gate="G$1" pin="P5"/>
+<wire x1="-120.015" y1="113.9825" x2="-106.9975" y2="113.9825" width="0.1524" layer="91"/>
+<wire x1="-106.9975" y1="113.9825" x2="-104.14" y2="116.84" width="0.1524" layer="91"/>
+<wire x1="-108.585" y1="140.0175" x2="-107.6325" y2="140.0175" width="0.1524" layer="91"/>
+<wire x1="-107.6325" y1="140.0175" x2="-106.68" y2="140.0175" width="0.1524" layer="91"/>
+<wire x1="-107.6325" y1="140.0175" x2="-107.6325" y2="183.8325" width="0.1524" layer="91"/>
+<wire x1="-107.6325" y1="183.8325" x2="-105.41" y2="186.055" width="0.1524" layer="91"/>
+<wire x1="-105.41" y1="186.055" x2="-33.02" y2="186.055" width="0.1524" layer="91"/>
+<wire x1="-33.02" y1="186.055" x2="-23.495" y2="195.58" width="0.1524" layer="91"/>
+<wire x1="-23.495" y1="195.58" x2="-2.54" y2="195.58" width="0.1524" layer="91"/>
+<label x="-120.3325" y="127.3175" size="1.778" layer="95"/>
+<label x="-119.6975" y="114.6175" size="1.778" layer="95"/>
 </segment>
 </net>
@@
 <wire x1="-99.695" y1="168.5925" x2="-96.2025" y2="172.085" width="0.1524" layer="91"/>
 <wire x1="-96.2025" y1="172.085" x2="-86.0425" y2="172.085" width="0.1524" layer="91"/>
-<pinref part="J1" gate="G$1" pin="P4"/>
-<wire x1="-120.015" y1="126.6825" x2="-113.665" y2="126.6825" width="0.1524" layer="91"/>
-<wire x1="-113.665" y1="126.6825" x2="-111.125" y2="129.2225" width="0.1524" layer="91"/>
-<wire x1="-111.125" y1="129.2225" x2="-111.125" y2="150.8125" width="0.1524" layer="91"/>
 <wire x1="-111.125" y1="150.8125" x2="-111.125" y2="163.195" width="0.1524" layer="91"/>
 <wire x1="-111.125" y1="163.195" x2="-111.125" y2="169.545" width="0.1524" layer="91"/>
 <wire x1="-111.125" y1="169.545" x2="-108.585" y2="172.085" width="0.1524" layer="91"/>
-<wire x1="-108.585" y1="172.085" x2="-105.7275" y2="172.085" width="0.1524" layer="91"/>
-<pinref part="J1" gate="G$1" pin="P5"/>
-<wire x1="-105.7275" y1="172.085" x2="-96.2025" y2="172.085" width="0.1524" layer="91"/>
-<wire x1="-120.015" y1="113.9825" x2="-106.9975" y2="113.9825" width="0.1524" layer="91"/>
-<wire x1="-106.9975" y1="113.9825" x2="-104.14" y2="116.84" width="0.1524" layer="91"/>
-<wire x1="-104.14" y1="116.84" x2="-104.14" y2="137.4775" width="0.1524" layer="91"/>
-<wire x1="-104.14" y1="137.4775" x2="-106.68" y2="140.0175" width="0.1524" layer="91"/>
-<wire x1="-106.68" y1="140.0175" x2="-106.68" y2="171.1325" width="0.1524" layer="91"/>
-<wire x1="-106.68" y1="171.1325" x2="-105.7275" y2="172.085" width="0.1524" layer="91"/>
+<wire x1="-108.585" y1="172.085" x2="-96.2025" y2="172.085" width="0.1524" layer="91"/>
 <pinref part="J1" gate="G$1" pin="GA"/>
 <wire x1="-120.015" y1="149.5425" x2="-112.395" y2="149.5425" width="0.1524" layer="91"/>
