File: STM32F107RC.ETH.sch (EAGLE design)
At the start: 35 parts, among them J1 HR911105A, Q1 8MHz, U1 LAN8720A-CP, U2 STM32F107RCT6, X1 CB3LV-3I-74M2500

Commit message: 6.11.18
Parts:
- added C10, C9: 104, resistor:C-EUC1206
Connections:
- net GND: now also C10.2, C9.2
- net VCC: now also C10.1, C9.1
Changed lines of the file:
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@@
 <part name="GND2" library="supply1" deviceset="GND" device=""/>
 <part name="GND3" library="supply1" deviceset="GND" device=""/>
+<part name="C9" library="resistor" deviceset="C-EU" device="C1206" value="104"/>
+<part name="GND4" library="supply1" deviceset="GND" device=""/>
+<part name="C10" library="resistor" deviceset="C-EU" device="C1206" value="104"/>
 </parts>
 <sheets>
@@
 <instance part="GND2" gate="1" x="7.62" y="126.365"/>
 <instance part="GND3" gate="1" x="149.5425" y="37.465"/>
+<instance part="C9" gate="G$1" x="148.2725" y="140.6525"/>
+<instance part="GND4" gate="1" x="148.2725" y="131.7625"/>
+<instance part="C10" gate="G$1" x="157.7975" y="140.6525"/>
 </instances>
 <busses>
@@
 <wire x1="141.605" y1="40.64" x2="149.5425" y2="40.64" width="0.1524" layer="91"/>
 <wire x1="149.5425" y1="40.64" x2="149.5425" y2="40.005" width="0.1524" layer="91"/>
+</segment>
+<segment>
+<pinref part="GND4" gate="1" pin="GND"/>
+<pinref part="C9" gate="G$1" pin="2"/>
+<wire x1="148.2725" y1="134.3025" x2="148.2725" y2="135.5725" width="0.1524" layer="91"/>
+<pinref part="C10" gate="G$1" pin="2"/>
+<wire x1="157.7975" y1="135.5725" x2="148.2725" y2="135.5725" width="0.1524" layer="91"/>
 </segment>
 </net>
@@
 <wire x1="137.16" y1="124.46" x2="140.6525" y2="124.46" width="0.1524" layer="91"/>
 <wire x1="140.6525" y1="124.46" x2="140.6525" y2="127" width="0.1524" layer="91"/>
-<wire x1="140.6525" y1="137.16" x2="140.6525" y2="146.3675" width="0.1524" layer="91"/>
+<wire x1="140.6525" y1="137.16" x2="140.6525" y2="143.1925" width="0.1524" layer="91"/>
+<wire x1="140.6525" y1="143.1925" x2="140.6525" y2="146.3675" width="0.1524" layer="91"/>
 <wire x1="140.6525" y1="146.3675" x2="77.7875" y2="146.3675" width="0.1524" layer="91"/>
-</segment>
-<segment>
+<pinref part="C9" gate="G$1" pin="1"/>
+<wire x1="148.2725" y1="143.1925" x2="140.6525" y2="143.1925" width="0.1524" layer="91"/>
+<pinref part="C10" gate="G$1" pin="1"/>
+<wire x1="148.2725" y1="143.1925" x2="157.7975" y2="143.1925" width="0.1524" layer="91"/>
+</segment>
+<segment>

Commit message: u 6.11.18
Parts:
- added C11: 105, resistor:C-EUC1206
- added J3: USB-MICROB, SparkFun-Connectors:USB-MICROB
- added J4: (no value), SparkFun-Connectors:M05LOCK_LONGPADS
- added JP3: (no value), jumper:JP1Q
- added U3: LM1117MP-3.3, LM1117MP-3.3:LM1117MP-3.3
- added X2: MSTBA6, con-phoenix-508:MSTBA6
Connections:
- new net N$23: C11.1, JP3.1, U3.IN
- net GND: now also C11.2, JP3.2, U3.ADJ/GND
- net VCC: now also U3.VOUT
Changed lines of the file:
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@@
 <setting verticaltext="up"/>
 </settings>
-<grid distance="12.5" unitdist="mil" unit="mil" style="lines" multiple="1" display="yes" altdistance="0.01" altunitdist="inch" altunit="inch"/>
+<grid distance="0.1" unitdist="inch" unit="inch" style="lines" multiple="1" display="no" altdistance="0.01" altunitdist="inch" altunit="inch"/>
 <layers>
 <layer number="1" name="Top" color="4" fill="1" visible="no" active="no"/>
@@
 <part name="GND4" library="supply1" deviceset="GND" device=""/>
 <part name="C10" library="resistor" deviceset="C-EU" device="C1206" value="104"/>
+<part name="U3" library="LM1117MP-3.3" deviceset="LM1117MP-3.3" device=""/>
+<part name="JP3" library="jumper" deviceset="JP1Q" device=""/>
+<part name="C11" library="resistor" deviceset="C-EU" device="C1206" value="105"/>
+<part name="X2" library="con-phoenix-508" deviceset="MSTBA6" device=""/>
+<part name="J3" library="SparkFun-Connectors" deviceset="USB" device="-MICROB"/>
+<part name="J4" library="SparkFun-Connectors" deviceset="M05" device="LOCK_LONGPADS"/>
 </parts>
 <sheets>
@@
 <instance part="GND4" gate="1" x="148.2725" y="131.7625"/>
 <instance part="C10" gate="G$1" x="157.7975" y="140.6525"/>
+<instance part="U3" gate="A" x="-55.88" y="227.0125"/>
+<instance part="JP3" gate="A" x="-86.995" y="224.79" rot="R180"/>
+<instance part="C11" gate="G$1" x="-79.0575" y="226.3775"/>
+<instance part="X2" gate="-1" x="38.1" y="-25.4" rot="R90"/>
+<instance part="X2" gate="-2" x="43.18" y="-25.4" rot="R90"/>
+<instance part="X2" gate="-3" x="48.26" y="-25.4" rot="R90"/>
+<instance part="X2" gate="-4" x="53.34" y="-25.4" rot="R90"/>
+<instance part="X2" gate="-5" x="58.42" y="-25.4" rot="R90"/>
+<instance part="X2" gate="-6" x="63.5" y="-25.4" rot="R90"/>
+<instance part="J3" gate="G$1" x="10.16" y="-25.4" rot="R270"/>
+<instance part="J4" gate="G$1" x="111.76" y="-15.24" rot="R90"/>
 </instances>
 <busses>
@@
 <wire x1="-103.505" y1="196.215" x2="-95.885" y2="203.835" width="0.1524" layer="91"/>
 <pinref part="JP2" gate="A" pin="2"/>
-<wire x1="-95.885" y1="203.835" x2="-64.4525" y2="203.835" width="0.1524" layer="91"/>
+<wire x1="-95.885" y1="203.835" x2="-79.0575" y2="203.835" width="0.1524" layer="91"/>
 <label x="-66.9925" y="204.1525" size="1.27" layer="95"/>
 <pinref part="C7" gate="G$1" pin="2"/>
+<wire x1="-79.0575" y1="203.835" x2="-64.4525" y2="203.835" width="0.1524" layer="91"/>
 <wire x1="-64.4525" y1="203.835" x2="-61.2775" y2="203.835" width="0.1524" layer="91"/>
 <wire x1="-56.8325" y1="196.215" x2="-62.865" y2="196.215" width="0.1524" layer="91"/>
 <wire x1="-62.865" y1="196.215" x2="-64.4525" y2="197.8025" width="0.1524" layer="91"/>
 <wire x1="-64.4525" y1="197.8025" x2="-64.4525" y2="203.835" width="0.1524" layer="91"/>
+<pinref part="JP3" gate="A" pin="2"/>
+<wire x1="-86.995" y1="217.17" x2="-86.995" y2="213.36" width="0.1524" layer="91"/>
+<wire x1="-86.995" y1="213.36" x2="-86.0425" y2="212.4075" width="0.1524" layer="91"/>
+<wire x1="-86.0425" y1="212.4075" x2="-79.0575" y2="212.4075" width="0.1524" layer="91"/>
+<wire x1="-79.0575" y1="212.4075" x2="-74.6125" y2="212.4075" width="0.1524" layer="91"/>
+<wire x1="-74.6125" y1="212.4075" x2="-73.66" y2="213.36" width="0.1524" layer="91"/>
+<pinref part="U3" gate="A" pin="ADJ/GND"/>
+<wire x1="-73.66" y1="213.36" x2="-73.66" y2="221.9325" width="0.1524" layer="91"/>
+<wire x1="-79.0575" y1="212.4075" x2="-79.0575" y2="203.835" width="0.1524" layer="91"/>
+<pinref part="C11" gate="G$1" pin="2"/>
+<wire x1="-79.0575" y1="221.2975" x2="-79.0575" y2="212.4075" width="0.1524" layer="91"/>
 </segment>
 <segment>
@@
 <pinref part="JP2" gate="A" pin="1"/>
 <wire x1="-46.0375" y1="203.835" x2="-42.2275" y2="203.835" width="0.1524" layer="91"/>
-<wire x1="-42.2275" y1="203.835" x2="-25.0825" y2="203.835" width="0.1524" layer="91"/>
+<wire x1="-42.2275" y1="203.835" x2="-30.1625" y2="203.835" width="0.1524" layer="91"/>
+<wire x1="-30.1625" y1="203.835" x2="-25.0825" y2="203.835" width="0.1524" layer="91"/>
 <wire x1="-25.0825" y1="203.835" x2="-13.0175" y2="215.9" width="0.1524" layer="91"/>
 <wire x1="-13.0175" y1="215.9" x2="0" y2="215.9" width="0.1524" layer="91"/>
@@
 <wire x1="-43.815" y1="196.215" x2="-42.2275" y2="197.8025" width="0.1524" layer="91"/>
 <wire x1="-42.2275" y1="197.8025" x2="-42.2275" y2="203.835" width="0.1524" layer="91"/>
+<pinref part="U3" gate="A" pin="VOUT"/>
+<wire x1="-38.1" y1="227.0125" x2="-31.4325" y2="227.0125" width="0.1524" layer="91"/>
+<wire x1="-31.4325" y1="227.0125" x2="-30.1625" y2="225.7425" width="0.1524" layer="91"/>
+<wire x1="-30.1625" y1="225.7425" x2="-30.1625" y2="203.835" width="0.1524" layer="91"/>
 </segment>
 <segment>
@@
 </segment>
 </net>
+<net name="N$23" class="0">
+<segment>
+<pinref part="JP3" gate="A" pin="1"/>
+<wire x1="-86.995" y1="232.41" x2="-86.995" y2="235.585" width="0.1524" layer="91"/>
+<wire x1="-86.995" y1="235.585" x2="-86.36" y2="236.22" width="0.1524" layer="91"/>
+<wire x1="-86.36" y1="236.22" x2="-79.0575" y2="236.22" width="0.1524" layer="91"/>
+<wire x1="-79.0575" y1="236.22" x2="-74.295" y2="236.22" width="0.1524" layer="91"/>
+<wire x1="-74.295" y1="236.22" x2="-73.66" y2="235.585" width="0.1524" layer="91"/>
+<pinref part="U3" gate="A" pin="IN"/>
+<wire x1="-73.66" y1="235.585" x2="-73.66" y2="227.0125" width="0.1524" layer="91"/>
+<pinref part="C11" gate="G$1" pin="1"/>
+<wire x1="-79.0575" y1="228.9175" x2="-79.0575" y2="236.22" width="0.1524" layer="91"/>
+</segment>
+</net>

Commit message: u 9-11-18
Parts:
- removed J4: (no value), SparkFun-Connectors:M05LOCK_LONGPADS
- added J5: (no value), SparkFun-Connectors:M06POLAR
Connections:
- removed net N$6: C1.1, R3.1, U2.NRST
- new net N$11: J5.1, U2.PB3
- new net NRST: C1.1, J5.5, R3.1, U2.NRST
- new net SWCLK: J5.4, U2.PA14
- new net SWDIO: J5.3, U2.PA13
- net GND: now also J5.6
- net VCC: now also J5.2
Changed lines of the file:
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@@
 <setting verticaltext="up"/>
 </settings>
-<grid distance="0.1" unitdist="inch" unit="inch" style="lines" multiple="1" display="no" altdistance="0.01" altunitdist="inch" altunit="inch"/>
+<grid distance="12.5" unitdist="mil" unit="mil" style="lines" multiple="1" display="yes" altdistance="0.01" altunitdist="inch" altunit="inch"/>
 <layers>
 <layer number="1" name="Top" color="4" fill="1" visible="no" active="no"/>
@@
 <part name="X2" library="con-phoenix-508" deviceset="MSTBA6" device=""/>
 <part name="J3" library="SparkFun-Connectors" deviceset="USB" device="-MICROB"/>
-<part name="J4" library="SparkFun-Connectors" deviceset="M05" device="LOCK_LONGPADS"/>
+<part name="J5" library="SparkFun-Connectors" deviceset="M06" device="POLAR"/>
+<part name="SUPPLY1" library="supply2" deviceset="VCC" device=""/>
+<part name="GND5" library="supply1" deviceset="GND" device=""/>
 </parts>
 <sheets>
@@
 <instance part="X2" gate="-6" x="63.5" y="-25.4" rot="R90"/>
 <instance part="J3" gate="G$1" x="10.16" y="-25.4" rot="R270"/>
-<instance part="J4" gate="G$1" x="111.76" y="-15.24" rot="R90"/>
+<instance part="J5" gate="G$1" x="45.72" y="50.8"/>
+<instance part="SUPPLY1" gate="G$1" x="68.8975" y="53.6575"/>
+<instance part="GND5" gate="1" x="53.975" y="64.77"/>
 </instances>
 <busses>
@@
 <wire x1="157.7975" y1="135.5725" x2="148.2725" y2="135.5725" width="0.1524" layer="91"/>
 </segment>
-</net>
-<net name="N$6" class="0">
+<segment>
+<pinref part="J5" gate="G$1" pin="6"/>
+<wire x1="50.8" y1="58.42" x2="51.1175" y2="58.42" width="0.1524" layer="91"/>
+<wire x1="51.1175" y1="58.42" x2="51.1175" y2="67.945" width="0.1524" layer="91"/>
+<pinref part="GND5" gate="1" pin="GND"/>
+<wire x1="51.1175" y1="67.945" x2="53.975" y2="67.945" width="0.1524" layer="91"/>
+<wire x1="53.975" y1="67.945" x2="53.975" y2="67.31" width="0.1524" layer="91"/>
+</segment>
+</net>
+<net name="NRST" class="0">
 <segment>
 <pinref part="U2" gate="A" pin="NRST"/>
@@
 <wire x1="60.96" y1="125.4125" x2="53.975" y2="129.2225" width="0.1524" layer="91"/>
 <wire x1="53.975" y1="125.4125" x2="60.96" y2="125.4125" width="0.1524" layer="91"/>
+<label x="69.215" y="117.1575" size="1.778" layer="95"/>
+</segment>
+<segment>
+<pinref part="J5" gate="G$1" pin="5"/>
+<wire x1="50.8" y1="55.88" x2="58.42" y2="55.88" width="0.1524" layer="91"/>
+<wire x1="58.42" y1="55.88" x2="58.42" y2="70.1675" width="0.1524" layer="91"/>
+<label x="60.325" y="60.96" size="1.778" layer="95" rot="R90"/>
 </segment>
 </net>
@@
 <wire x1="-112.0775" y1="162.2425" x2="-111.125" y2="163.195" width="0.1524" layer="91"/>
 </segment>
+<segment>
+<pinref part="J5" gate="G$1" pin="2"/>
+<pinref part="SUPPLY1" gate="G$1" pin="VCC"/>
+<wire x1="50.8" y1="48.26" x2="68.8975" y2="48.26" width="0.1524" layer="91"/>
+<wire x1="68.8975" y1="48.26" x2="68.8975" y2="51.1175" width="0.1524" layer="91"/>
+</segment>
 </net>
 <net name="N$16" class="0">
@@
 </segment>
 </net>
+<net name="N$11" class="0">
+<segment>
+<pinref part="J5" gate="G$1" pin="1"/>
+<wire x1="50.8" y1="45.72" x2="71.755" y2="45.72" width="0.1524" layer="91"/>
+<wire x1="71.755" y1="45.72" x2="71.755" y2="60.96" width="0.1524" layer="91"/>
+<pinref part="U2" gate="A" pin="PB3"/>
+<wire x1="71.755" y1="60.96" x2="81.28" y2="60.96" width="0.1524" layer="91"/>
+</segment>
+</net>
+<net name="SWDIO" class="0">
+<segment>
+<pinref part="U2" gate="A" pin="PA13"/>
+<wire x1="81.28" y1="78.74" x2="66.675" y2="78.74" width="0.1524" layer="91"/>
+<wire x1="66.675" y1="78.74" x2="66.675" y2="50.8" width="0.1524" layer="91"/>
+<pinref part="J5" gate="G$1" pin="3"/>
+<wire x1="66.675" y1="50.8" x2="50.8" y2="50.8" width="0.1524" layer="91"/>
+<label x="68.8975" y="64.135" size="1.778" layer="95" rot="R90"/>
+</segment>
+</net>
+<net name="SWCLK" class="0">
+<segment>
+<pinref part="U2" gate="A" pin="PA14"/>
+<wire x1="81.28" y1="76.2" x2="63.1825" y2="76.2" width="0.1524" layer="91"/>
+<wire x1="63.1825" y1="76.2" x2="63.1825" y2="53.34" width="0.1524" layer="91"/>
+<pinref part="J5" gate="G$1" pin="4"/>
+<wire x1="63.1825" y1="53.34" x2="50.8" y2="53.34" width="0.1524" layer="91"/>
+<label x="65.405" y="64.4525" size="1.778" layer="95" rot="R90"/>
+</segment>
+</net>

Commit message: u 10-11-18
Parts:
- removed J3: USB-MICROB, SparkFun-Connectors:USB-MICROB
- added J4: USB-MICROB", SparkFun-Connectors:USB-MICROB"
Connections:
- net N$11 renamed SWO
- new net N$11: J4.D-, U2.PA11
- new net N$28: J4.D+, U2.PA12
- new net N$6: J4.VBUS, U2.PA9
- net GND: now also J4.GND
Changed lines of the file:
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@@
 <part name="C11" library="resistor" deviceset="C-EU" device="C1206" value="105"/>
 <part name="X2" library="con-phoenix-508" deviceset="MSTBA6" device=""/>
-<part name="J3" library="SparkFun-Connectors" deviceset="USB" device="-MICROB"/>
 <part name="J5" library="SparkFun-Connectors" deviceset="M06" device="POLAR"/>
 <part name="SUPPLY1" library="supply2" deviceset="VCC" device=""/>
 <part name="GND5" library="supply1" deviceset="GND" device=""/>
+<part name="J4" library="SparkFun-Connectors" deviceset="USB-MICROB" device="&quot;"/>
 </parts>
 <sheets>
@@
 <instance part="X2" gate="-5" x="58.42" y="-25.4" rot="R90"/>
 <instance part="X2" gate="-6" x="63.5" y="-25.4" rot="R90"/>
-<instance part="J3" gate="G$1" x="10.16" y="-25.4" rot="R270"/>
 <instance part="J5" gate="G$1" x="45.72" y="50.8"/>
 <instance part="SUPPLY1" gate="G$1" x="68.8975" y="53.6575"/>
 <instance part="GND5" gate="1" x="53.975" y="64.77"/>
+<instance part="J4" gate="G$1" x="41.91" y="76.835" rot="R180"/>
 </instances>
 <busses>
@@
 <wire x1="51.1175" y1="67.945" x2="53.975" y2="67.945" width="0.1524" layer="91"/>
 <wire x1="53.975" y1="67.945" x2="53.975" y2="67.31" width="0.1524" layer="91"/>
+<pinref part="J4" gate="G$1" pin="GND"/>
+<wire x1="46.99" y1="69.215" x2="50.4825" y2="69.215" width="0.1524" layer="91"/>
+<wire x1="50.4825" y1="69.215" x2="51.1175" y2="68.58" width="0.1524" layer="91"/>
+<wire x1="51.1175" y1="68.58" x2="51.1175" y2="67.945" width="0.1524" layer="91"/>
 </segment>
 </net>
@@
 </segment>
 </net>
-<net name="N$11" class="0">
+<net name="SWO" class="0">
 <segment>
 <pinref part="J5" gate="G$1" pin="1"/>
@@
 <pinref part="U2" gate="A" pin="PB3"/>
 <wire x1="71.755" y1="60.96" x2="81.28" y2="60.96" width="0.1524" layer="91"/>
+<label x="73.9775" y="47.625" size="1.778" layer="95" rot="R90"/>
 </segment>
 </net>
@@
 </segment>
 </net>
+<net name="N$6" class="0">
+<segment>
+<pinref part="U2" gate="A" pin="PA9"/>
+<wire x1="81.28" y1="88.9" x2="53.0225" y2="88.9" width="0.1524" layer="91"/>
+<wire x1="53.0225" y1="88.9" x2="51.1175" y2="86.995" width="0.1524" layer="91"/>
+<wire x1="51.1175" y1="86.995" x2="51.1175" y2="80.3275" width="0.1524" layer="91"/>
+<wire x1="51.1175" y1="80.3275" x2="50.165" y2="79.375" width="0.1524" layer="91"/>
+<pinref part="J4" gate="G$1" pin="VBUS"/>
+<wire x1="50.165" y1="79.375" x2="46.99" y2="79.375" width="0.1524" layer="91"/>
+</segment>
+</net>
+<net name="N$11" class="0">
+<segment>
+<pinref part="U2" gate="A" pin="PA11"/>
+<wire x1="81.28" y1="83.82" x2="54.9275" y2="83.82" width="0.1524" layer="91"/>
+<wire x1="54.9275" y1="83.82" x2="53.6575" y2="82.55" width="0.1524" layer="91"/>
+<wire x1="53.6575" y1="82.55" x2="53.6575" y2="77.7875" width="0.1524" layer="91"/>
+<wire x1="53.6575" y1="77.7875" x2="52.705" y2="76.835" width="0.1524" layer="91"/>
+<pinref part="J4" gate="G$1" pin="D-"/>
+<wire x1="52.705" y1="76.835" x2="46.99" y2="76.835" width="0.1524" layer="91"/>
+</segment>
+</net>
+<net name="N$28" class="0">
+<segment>
+<pinref part="U2" gate="A" pin="PA12"/>
+<wire x1="81.28" y1="81.28" x2="56.515" y2="81.28" width="0.1524" layer="91"/>
+<wire x1="56.515" y1="81.28" x2="55.5625" y2="80.3275" width="0.1524" layer="91"/>
+<wire x1="55.5625" y1="80.3275" x2="55.5625" y2="75.2475" width="0.1524" layer="91"/>
+<wire x1="55.5625" y1="75.2475" x2="54.61" y2="74.295" width="0.1524" layer="91"/>
+<pinref part="J4" gate="G$1" pin="D+"/>
+<wire x1="54.61" y1="74.295" x2="46.99" y2="74.295" width="0.1524" layer="91"/>
+</segment>
+</net>
