File: STM32F107RC.ETH.sch (EAGLE design)
At the start: 43 parts, among them J1 HR911105A, J4 USB-MICROB", Q1 8MHz, U1 LAN8720A-CP, U2 STM32F107RCT6, U3 LM1117MP-3.3, X1 CB3LV-3I-74M2500, X2 MSTBA6

Commit message: u 10-11-18 added USB OPTO INPUT;
Parts:
- added LED1, LED2, LED3: (no value), led:LEDCHIPLED_0805
- added R19, R20, R21: (no value), SparkFun-Resistors:RESISTOR0805-RES
- added U4: TLP281-4GB(F), TLP281-4GB_F_:TLP281-4GB(F)
Connections:
- new net N$29: R19.1, X2-1.1
- new net N$30: R20.1, X2-2.1
- new net N$31: R21.1, X2-3.1
- new net N$32: LED1.C, R19.2
- new net N$33: LED2.C, R20.2
- new net N$34: LED3.C, R21.2
- new net N$35: LED1.A, U4.C1
- new net N$36: LED2.A, U4.C2
- new net N$37: LED3.A, U4.C3
- new net N$38: U4.A1, U4.A2, U4.A3
Other:
- moved on the sheet: X2-1, X2-2, X2-3, X2-4, X2-5, X2-6
Changed lines of the file:
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@@
 <part name="GND5" library="supply1" deviceset="GND" device=""/>
 <part name="J4" library="SparkFun-Connectors" deviceset="USB-MICROB" device="&quot;"/>
+<part name="U4" library="TLP281-4GB_F_" deviceset="TLP281-4GB(F)" device=""/>
+<part name="LED1" library="led" deviceset="LED" device="CHIPLED_0805"/>
+<part name="R19" library="SparkFun-Resistors" deviceset="RESISTOR" device="0805-RES"/>
+<part name="R20" library="SparkFun-Resistors" deviceset="RESISTOR" device="0805-RES"/>
+<part name="R21" library="SparkFun-Resistors" deviceset="RESISTOR" device="0805-RES"/>
+<part name="LED2" library="led" deviceset="LED" device="CHIPLED_0805"/>
+<part name="LED3" library="led" deviceset="LED" device="CHIPLED_0805"/>
 </parts>
 <sheets>
@@
 <instance part="JP3" gate="A" x="-86.995" y="224.79" rot="R180"/>
 <instance part="C11" gate="G$1" x="-79.0575" y="226.3775"/>
-<instance part="X2" gate="-1" x="38.1" y="-25.4" rot="R90"/>
-<instance part="X2" gate="-2" x="43.18" y="-25.4" rot="R90"/>
-<instance part="X2" gate="-3" x="48.26" y="-25.4" rot="R90"/>
-<instance part="X2" gate="-4" x="53.34" y="-25.4" rot="R90"/>
-<instance part="X2" gate="-5" x="58.42" y="-25.4" rot="R90"/>
-<instance part="X2" gate="-6" x="63.5" y="-25.4" rot="R90"/>
+<instance part="X2" gate="-1" x="-148.59" y="-17.4625"/>
+<instance part="X2" gate="-2" x="-148.59" y="-22.5425"/>
+<instance part="X2" gate="-3" x="-148.59" y="-27.6225"/>
+<instance part="X2" gate="-4" x="-148.59" y="-32.7025"/>
+<instance part="X2" gate="-5" x="-148.59" y="-37.7825"/>
+<instance part="X2" gate="-6" x="-148.59" y="-42.8625"/>
 <instance part="J5" gate="G$1" x="45.72" y="50.8"/>
 <instance part="SUPPLY1" gate="G$1" x="68.8975" y="53.6575"/>
 <instance part="GND5" gate="1" x="53.975" y="64.77"/>
 <instance part="J4" gate="G$1" x="41.91" y="76.835" rot="R180"/>
+<instance part="U4" gate="G$1" x="-84.1375" y="-29.5275"/>
+<instance part="LED1" gate="G$1" x="-120.65" y="-17.4625" rot="R270"/>
+<instance part="R19" gate="G$1" x="-134.3025" y="-17.4625"/>
+<instance part="R20" gate="G$1" x="-134.3025" y="-22.5425"/>
+<instance part="R21" gate="G$1" x="-134.3025" y="-27.6225"/>
+<instance part="LED2" gate="G$1" x="-120.65" y="-22.5425" rot="R270"/>
+<instance part="LED3" gate="G$1" x="-120.65" y="-27.6225" rot="R270"/>
 </instances>
 <busses>
@@
 </segment>
 </net>
+<net name="N$29" class="0">
+<segment>
+<pinref part="X2" gate="-1" pin="1"/>
+<pinref part="R19" gate="G$1" pin="1"/>
+<wire x1="-143.51" y1="-17.4625" x2="-139.3825" y2="-17.4625" width="0.1524" layer="91"/>
+</segment>
+</net>
+<net name="N$30" class="0">
+<segment>
+<pinref part="X2" gate="-2" pin="1"/>
+<pinref part="R20" gate="G$1" pin="1"/>
+<wire x1="-143.51" y1="-22.5425" x2="-139.3825" y2="-22.5425" width="0.1524" layer="91"/>
+</segment>
+</net>
+<net name="N$31" class="0">
+<segment>
+<pinref part="R21" gate="G$1" pin="1"/>
+<pinref part="X2" gate="-3" pin="1"/>
+<wire x1="-139.3825" y1="-27.6225" x2="-143.51" y2="-27.6225" width="0.1524" layer="91"/>
+</segment>
+</net>
+<net name="N$32" class="0">
+<segment>
+<pinref part="R19" gate="G$1" pin="2"/>
+<pinref part="LED1" gate="G$1" pin="C"/>
+<wire x1="-129.2225" y1="-17.4625" x2="-125.73" y2="-17.4625" width="0.1524" layer="91"/>
+</segment>
+</net>
+<net name="N$33" class="0">
+<segment>
+<pinref part="LED2" gate="G$1" pin="C"/>
+<pinref part="R20" gate="G$1" pin="2"/>
+<wire x1="-125.73" y1="-22.5425" x2="-129.2225" y2="-22.5425" width="0.1524" layer="91"/>
+</segment>
+</net>
+<net name="N$34" class="0">
+<segment>
+<pinref part="R21" gate="G$1" pin="2"/>
+<pinref part="LED3" gate="G$1" pin="C"/>
+<wire x1="-129.2225" y1="-27.6225" x2="-125.73" y2="-27.6225" width="0.1524" layer="91"/>
+</segment>
+</net>
+<net name="N$35" class="0">
+<segment>
+<pinref part="LED1" gate="G$1" pin="A"/>
+<pinref part="U4" gate="G$1" pin="C1"/>
+<wire x1="-118.11" y1="-17.4625" x2="-96.2025" y2="-17.4625" width="0.1524" layer="91"/>
+<wire x1="-96.2025" y1="-17.4625" x2="-94.2975" y2="-19.3675" width="0.1524" layer="91"/>
+</segment>
+</net>
+<net name="N$36" class="0">
+<segment>
+<pinref part="LED2" gate="G$1" pin="A"/>
+<wire x1="-118.11" y1="-22.5425" x2="-104.775" y2="-22.5425" width="0.1524" layer="91"/>
+<wire x1="-104.775" y1="-22.5425" x2="-103.1875" y2="-24.13" width="0.1524" layer="91"/>
+<wire x1="-103.1875" y1="-24.13" x2="-103.1875" y2="-28.2575" width="0.1524" layer="91"/>
+<wire x1="-103.1875" y1="-28.2575" x2="-101.9175" y2="-29.5275" width="0.1524" layer="91"/>
+<pinref part="U4" gate="G$1" pin="C2"/>
+<wire x1="-101.9175" y1="-29.5275" x2="-94.2975" y2="-29.5275" width="0.1524" layer="91"/>
+</segment>
+</net>
+<net name="N$37" class="0">
+<segment>
+<pinref part="LED3" gate="G$1" pin="A"/>
+<wire x1="-118.11" y1="-27.6225" x2="-106.045" y2="-27.6225" width="0.1524" layer="91"/>
+<wire x1="-106.045" y1="-27.6225" x2="-105.0925" y2="-28.575" width="0.1524" layer="91"/>
+<wire x1="-105.0925" y1="-28.575" x2="-105.0925" y2="-38.4175" width="0.1524" layer="91"/>
+<wire x1="-105.0925" y1="-38.4175" x2="-103.8225" y2="-39.6875" width="0.1524" layer="91"/>
+<pinref part="U4" gate="G$1" pin="C3"/>
+<wire x1="-103.8225" y1="-39.6875" x2="-94.2975" y2="-39.6875" width="0.1524" layer="91"/>
+</segment>
+</net>
+<net name="N$38" class="0">
+<segment>
+<pinref part="U4" gate="G$1" pin="A3"/>
+<wire x1="-94.2975" y1="-32.0675" x2="-96.8375" y2="-32.0675" width="0.1524" layer="91"/>
+<wire x1="-96.8375" y1="-32.0675" x2="-97.79" y2="-31.115" width="0.1524" layer="91"/>
+<wire x1="-97.79" y1="-31.115" x2="-97.79" y2="-20.955" width="0.1524" layer="91"/>
+<pinref part="U4" gate="G$1" pin="A1"/>
+<wire x1="-97.79" y1="-20.955" x2="-97.79" y2="-10.795" width="0.1524" layer="91"/>
+<wire x1="-97.79" y1="-10.795" x2="-97.79" y2="-8.5725" width="0.1524" layer="91"/>
+<wire x1="-94.2975" y1="-11.7475" x2="-96.8375" y2="-11.7475" width="0.1524" layer="91"/>
+<wire x1="-96.8375" y1="-11.7475" x2="-97.79" y2="-10.795" width="0.1524" layer="91"/>
+<pinref part="U4" gate="G$1" pin="A2"/>
+<wire x1="-94.2975" y1="-21.9075" x2="-96.8375" y2="-21.9075" width="0.1524" layer="91"/>
+<wire x1="-96.8375" y1="-21.9075" x2="-97.79" y2="-20.955" width="0.1524" layer="91"/>
+</segment>
+</net>

Commit message: u 12-11-18
Parts:
- added LED4, LED5: (no value), led:LEDCHIPLED_0805
- added R22, R23: (no value), SparkFun-Resistors:RESISTOR0805-RES
- added U5: TLP281-4GB(F), TLP281-4GB_F_:TLP281-4GB(F)
- added X3: MSTBA6, con-phoenix-508:MSTBA6
Connections:
- new net N$39: R22.1, X2-4.1
- new net N$40: LED4.C, R22.2
- new net N$41: LED4.A, U4.C4
- new net N$45: R23.1, X2-5.1
- new net N$46: LED5.C, R23.2
- new net N$47: LED5.A, U5.C1
- net N$38: now also U4.A4, U5.A1, X2-6.1
Changed lines of the file:
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@@
 <part name="LED2" library="led" deviceset="LED" device="CHIPLED_0805"/>
 <part name="LED3" library="led" deviceset="LED" device="CHIPLED_0805"/>
+<part name="LED4" library="led" deviceset="LED" device="CHIPLED_0805"/>
+<part name="R22" library="SparkFun-Resistors" deviceset="RESISTOR" device="0805-RES"/>
+<part name="U5" library="TLP281-4GB_F_" deviceset="TLP281-4GB(F)" device=""/>
+<part name="R23" library="SparkFun-Resistors" deviceset="RESISTOR" device="0805-RES"/>
+<part name="LED5" library="led" deviceset="LED" device="CHIPLED_0805"/>
+<part name="X3" library="con-phoenix-508" deviceset="MSTBA6" device=""/>
 </parts>
 <sheets>
@@
 <instance part="LED2" gate="G$1" x="-120.65" y="-22.5425" rot="R270"/>
 <instance part="LED3" gate="G$1" x="-120.65" y="-27.6225" rot="R270"/>
+<instance part="LED4" gate="G$1" x="-120.65" y="-32.7025" rot="R270"/>
+<instance part="R22" gate="G$1" x="-134.3025" y="-32.7025"/>
+<instance part="U5" gate="G$1" x="-84.1375" y="-77.7875"/>
+<instance part="R23" gate="G$1" x="-134.3025" y="-37.7825"/>
+<instance part="LED5" gate="G$1" x="-120.65" y="-37.7825" rot="R270"/>
+<instance part="X3" gate="-1" x="260.6675" y="-44.7675" rot="R180"/>
+<instance part="X3" gate="-2" x="260.6675" y="-39.6875" rot="R180"/>
+<instance part="X3" gate="-3" x="260.6675" y="-34.6075" rot="R180"/>
+<instance part="X3" gate="-4" x="260.6675" y="-29.5275" rot="R180"/>
+<instance part="X3" gate="-5" x="260.6675" y="-24.4475" rot="R180"/>
+<instance part="X3" gate="-6" x="260.6675" y="-19.3675" rot="R180"/>
 </instances>
 <busses>
@@
 <wire x1="-94.2975" y1="-21.9075" x2="-96.8375" y2="-21.9075" width="0.1524" layer="91"/>
 <wire x1="-96.8375" y1="-21.9075" x2="-97.79" y2="-20.955" width="0.1524" layer="91"/>
-</segment>
-</net>
+<pinref part="U4" gate="G$1" pin="A4"/>
+<wire x1="-94.2975" y1="-42.2275" x2="-96.52" y2="-42.2275" width="0.1524" layer="91"/>
+<wire x1="-96.52" y1="-42.2275" x2="-97.79" y2="-40.9575" width="0.1524" layer="91"/>
+<wire x1="-97.79" y1="-40.9575" x2="-97.79" y2="-31.115" width="0.1524" layer="91"/>
+<pinref part="U5" gate="G$1" pin="A1"/>
+<wire x1="-94.2975" y1="-60.0075" x2="-96.8375" y2="-60.0075" width="0.1524" layer="91"/>
+<wire x1="-96.8375" y1="-60.0075" x2="-97.79" y2="-58.7375" width="0.1524" layer="91"/>
+<wire x1="-97.79" y1="-58.7375" x2="-97.79" y2="-40.9575" width="0.1524" layer="91"/>
+<pinref part="X2" gate="-6" pin="1"/>
+<wire x1="-143.51" y1="-42.8625" x2="-141.2875" y2="-45.085" width="0.1524" layer="91"/>
+<wire x1="-141.2875" y1="-45.085" x2="-118.11" y2="-45.085" width="0.1524" layer="91"/>
+<wire x1="-118.11" y1="-45.085" x2="-114.935" y2="-41.91" width="0.1524" layer="91"/>
+<wire x1="-114.935" y1="-41.91" x2="-114.935" y2="-9.525" width="0.1524" layer="91"/>
+<wire x1="-114.935" y1="-9.525" x2="-113.665" y2="-8.255" width="0.1524" layer="91"/>
+<wire x1="-113.665" y1="-8.255" x2="-98.1075" y2="-8.255" width="0.1524" layer="91"/>
+<wire x1="-98.1075" y1="-8.255" x2="-97.79" y2="-8.5725" width="0.1524" layer="91"/>
+</segment>
+</net>
+<net name="N$39" class="0">
+<segment>
+<pinref part="X2" gate="-4" pin="1"/>
+<pinref part="R22" gate="G$1" pin="1"/>
+<wire x1="-143.51" y1="-32.7025" x2="-139.3825" y2="-32.7025" width="0.1524" layer="91"/>
+</segment>
+</net>
+<net name="N$40" class="0">
+<segment>
+<pinref part="R22" gate="G$1" pin="2"/>
+<pinref part="LED4" gate="G$1" pin="C"/>
+<wire x1="-129.2225" y1="-32.7025" x2="-125.73" y2="-32.7025" width="0.1524" layer="91"/>
+</segment>
+</net>
+<net name="N$41" class="0">
+<segment>
+<pinref part="LED4" gate="G$1" pin="A"/>
+<wire x1="-118.11" y1="-32.7025" x2="-108.2675" y2="-32.7025" width="0.1524" layer="91"/>
+<wire x1="-108.2675" y1="-32.7025" x2="-107.315" y2="-33.655" width="0.1524" layer="91"/>
+<wire x1="-107.315" y1="-33.655" x2="-107.315" y2="-48.5775" width="0.1524" layer="91"/>
+<wire x1="-107.315" y1="-48.5775" x2="-106.045" y2="-49.8475" width="0.1524" layer="91"/>
+<pinref part="U4" gate="G$1" pin="C4"/>
+<wire x1="-106.045" y1="-49.8475" x2="-94.2975" y2="-49.8475" width="0.1524" layer="91"/>
+</segment>
+</net>
+<net name="N$45" class="0">
+<segment>
+<pinref part="X2" gate="-5" pin="1"/>
+<pinref part="R23" gate="G$1" pin="1"/>
+<wire x1="-143.51" y1="-37.7825" x2="-139.3825" y2="-37.7825" width="0.1524" layer="91"/>
+</segment>
+</net>
+<net name="N$46" class="0">
+<segment>
+<pinref part="R23" gate="G$1" pin="2"/>
+<pinref part="LED5" gate="G$1" pin="C"/>
+<wire x1="-129.2225" y1="-37.7825" x2="-125.73" y2="-37.7825" width="0.1524" layer="91"/>
+</segment>
+</net>
+<net name="N$47" class="0">
+<segment>
+<pinref part="LED5" gate="G$1" pin="A"/>
+<wire x1="-118.11" y1="-37.7825" x2="-109.855" y2="-37.7825" width="0.1524" layer="91"/>
+<wire x1="-109.855" y1="-37.7825" x2="-109.22" y2="-38.4175" width="0.1524" layer="91"/>
+<wire x1="-109.22" y1="-38.4175" x2="-109.22" y2="-64.4525" width="0.1524" layer="91"/>
+<pinref part="U5" gate="G$1" pin="C1"/>
+<wire x1="-109.22" y1="-64.4525" x2="-106.045" y2="-67.6275" width="0.1524" layer="91"/>
+<wire x1="-106.045" y1="-67.6275" x2="-94.2975" y2="-67.6275" width="0.1524" layer="91"/>
+</segment>
+</net>

Commit message: omron relay library added. 12-11-18
Parts:
- added U$1: OMRON-RELAY-G5NB, omron-G5NB-1A-E:OMRON-RELAY-G5NB
Changed lines of the file:
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@@
 <setting verticaltext="up"/>
 </settings>
-<grid distance="12.5" unitdist="mil" unit="mil" style="lines" multiple="1" display="yes" altdistance="0.01" altunitdist="inch" altunit="inch"/>
+<grid distance="0.1" unitdist="inch" unit="inch" style="lines" multiple="1" display="no" altdistance="0.01" altunitdist="inch" altunit="inch"/>
 <layers>
 <layer number="1" name="Top" color="4" fill="1" visible="no" active="no"/>
@@
 <part name="LED5" library="led" deviceset="LED" device="CHIPLED_0805"/>
 <part name="X3" library="con-phoenix-508" deviceset="MSTBA6" device=""/>
+<part name="U$1" library="omron-G5NB-1A-E" deviceset="OMRON-RELAY-G5NB" device=""/>
 </parts>
 <sheets>
@@
 <instance part="X3" gate="-5" x="260.6675" y="-24.4475" rot="R180"/>
 <instance part="X3" gate="-6" x="260.6675" y="-19.3675" rot="R180"/>
+<instance part="U$1" gate="G$1" x="203.2" y="91.44"/>
 </instances>
 <busses>
