File: STM32F107RC.ETH.sch (EAGLE design)
At the start: 57 parts, among them J1 HR911105A, J4 USB-MICROB", Q1 8MHz, U1 LAN8720A-CP, U2 STM32F107RCT6, U3 LM1117MP-3.3, U4 TLP281-4GB(F), U5 TLP281-4GB(F), X1 CB3LV-3I-74M2500, X2 MSTBA6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

Commit message: U01.12.18
Parts:
- added IC1: LM358, SparkFun-AnalogIC:LM358
Other:
- moved on the sheet: X3-1, X3-2, X3-3, X3-4, X3-5, X3-6
Changed lines of the file:
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@@
 <part name="X3" library="con-phoenix-508" deviceset="MSTBA6" device=""/>
 <part name="U$1" library="omron-G5NB-1A-E" deviceset="OMRON-RELAY-G5NB" device=""/>
+<part name="IC1" library="SparkFun-AnalogIC" deviceset="LM358" device=""/>
 </parts>
 <sheets>
@@
 <instance part="R23" gate="G$1" x="-134.3025" y="-37.7825"/>
 <instance part="LED5" gate="G$1" x="-120.65" y="-37.7825" rot="R270"/>
-<instance part="X3" gate="-1" x="260.6675" y="-44.7675" rot="R180"/>
-<instance part="X3" gate="-2" x="260.6675" y="-39.6875" rot="R180"/>
-<instance part="X3" gate="-3" x="260.6675" y="-34.6075" rot="R180"/>
-<instance part="X3" gate="-4" x="260.6675" y="-29.5275" rot="R180"/>
-<instance part="X3" gate="-5" x="260.6675" y="-24.4475" rot="R180"/>
-<instance part="X3" gate="-6" x="260.6675" y="-19.3675" rot="R180"/>
+<instance part="X3" gate="-1" x="-192.0875" y="303.8475"/>
+<instance part="X3" gate="-2" x="-192.0875" y="298.7675"/>
+<instance part="X3" gate="-3" x="-192.0875" y="293.6875"/>
+<instance part="X3" gate="-4" x="-192.0875" y="288.6075"/>
+<instance part="X3" gate="-5" x="-192.0875" y="283.5275"/>
+<instance part="X3" gate="-6" x="-192.0875" y="278.4475"/>
 <instance part="U$1" gate="G$1" x="203.2" y="91.44"/>
+<instance part="IC1" gate="G1" x="-160.02" y="299.72" rot="MR180"/>
+<instance part="IC1" gate="G2" x="-157.48" y="279.4"/>
 </instances>
 <busses>

Commit message: uu
Parts:
- removed IC1: LM358, SparkFun-AnalogIC:LM358
- added C12, C14: 0.1uF, SparkFun-Capacitors:0.1UF-25V-5%(0603)
- added IC2: LM358, SparkFun-AnalogIC:LM358
- added R24, R30: 0.3, SparkFun-Resistors:0.3OHM-1/8W-1%(0805)
- added R25, R26, R27, R28, R29, R32, R33, R34, R35, R36: 1K, SparkFun-Resistors:1KOHM-1/4W-1%(PTH)
- added SJ1, SJ2: (no value), jumper:SJ2W
Connections:
- new net N$44: C12.2, IC2G2.-IN, R25.1, R26.2, R29.1
- new net N$48: IC2G2.+IN, R27.2, R28.1
- new net N$49: IC2G2.OUT, R25.2, R30.1
- new net N$50: R28.2, SJ2.1
- new net N$51: R29.2, SJ2.3
- new net N$55: IC2G1.-IN, R32.1, R34.2, R35.1
- new net N$56: C14.2, IC2G1.+IN, R33.2, R36.1
- new net N$58: IC2G1.OUT, R24.1, R32.2
- new net N$60: R35.2, SJ1.1
- new net N$61: R36.2, SJ1.3
- net GND: now also C12.1, C14.1, IC2G1.V-, R26.1, R27.1, R33.1, R34.1

Commit message: gg
Parts:
- added R31, R37: 1K, SparkFun-Resistors:1KOHM-1/4W-1%(PTH)
Connections:
- new net +5V: IC2G1.V+, R31.2, R37.2
Changed lines of the file:
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@@
 <part name="SJ2" library="jumper" deviceset="SJ2W" device=""/>
 <part name="R30" library="SparkFun-Resistors" deviceset="0.3OHM-1/8W-1%(0805)" device="" value="0.3"/>
+<part name="P+1" library="supply1" deviceset="+5V" device=""/>
+<part name="R31" library="SparkFun-Resistors" deviceset="1KOHM-1/4W-1%(PTH)" device="" value="1K"/>
+<part name="R37" library="SparkFun-Resistors" deviceset="1KOHM-1/4W-1%(PTH)" device="" value="1K"/>
 </parts>
 <sheets>
@@
 <instance part="R30" gate="G$1" x="-70.1675" y="302.5775"/>
 <instance part="IC2" gate="G2" x="-90.17" y="302.5775"/>
+<instance part="P+1" gate="1" x="-93.98" y="383.54"/>
+<instance part="R31" gate="G$1" x="-112.7125" y="378.1425"/>
+<instance part="R37" gate="G$1" x="-113.03" y="386.3975"/>
 </instances>
 <busses>
@@
 </segment>
 </net>
+<net name="+5V" class="0">
+<segment>
+<pinref part="IC2" gate="G1" pin="V+"/>
+<wire x1="-94.2975" y1="359.7275" x2="-94.2975" y2="361.6325" width="0.1524" layer="91"/>
+<wire x1="-94.2975" y1="361.6325" x2="-93.6625" y2="362.2675" width="0.1524" layer="91"/>
+<wire x1="-93.6625" y1="362.2675" x2="-84.1375" y2="362.2675" width="0.1524" layer="91"/>
+<wire x1="-84.1375" y1="362.2675" x2="-83.185" y2="363.22" width="0.1524" layer="91"/>
+<wire x1="-83.185" y1="363.22" x2="-83.185" y2="378.1425" width="0.1524" layer="91"/>
+<wire x1="-83.185" y1="378.1425" x2="-84.1375" y2="379.095" width="0.1524" layer="91"/>
+<wire x1="-84.1375" y1="379.095" x2="-93.345" y2="379.095" width="0.1524" layer="91"/>
+<wire x1="-93.345" y1="379.095" x2="-93.98" y2="379.73" width="0.1524" layer="91"/>
+<pinref part="P+1" gate="1" pin="+5V"/>
+<wire x1="-93.98" y1="379.73" x2="-93.98" y2="381" width="0.1524" layer="91"/>
+<pinref part="R37" gate="G$1" pin="2"/>
+<wire x1="-107.95" y1="386.3975" x2="-106.3625" y2="386.3975" width="0.1524" layer="91"/>
+<wire x1="-106.3625" y1="386.3975" x2="-105.41" y2="385.445" width="0.1524" layer="91"/>
+<wire x1="-105.41" y1="385.445" x2="-105.41" y2="382.5875" width="0.1524" layer="91"/>
+<wire x1="-105.41" y1="382.5875" x2="-105.41" y2="379.095" width="0.1524" layer="91"/>
+<wire x1="-105.41" y1="379.095" x2="-106.3625" y2="378.1425" width="0.1524" layer="91"/>
+<pinref part="R31" gate="G$1" pin="2"/>
+<wire x1="-106.3625" y1="378.1425" x2="-107.6325" y2="378.1425" width="0.1524" layer="91"/>
+<wire x1="-105.41" y1="382.5875" x2="-103.1875" y2="382.5875" width="0.1524" layer="91"/>
+<wire x1="-103.1875" y1="382.5875" x2="-102.5525" y2="381.9525" width="0.1524" layer="91"/>
+<wire x1="-102.5525" y1="381.9525" x2="-102.5525" y2="375.285" width="0.1524" layer="91"/>
+<wire x1="-102.5525" y1="375.285" x2="-101.9175" y2="374.65" width="0.1524" layer="91"/>
+<wire x1="-101.9175" y1="374.65" x2="-94.615" y2="374.65" width="0.1524" layer="91"/>
+<wire x1="-94.615" y1="374.65" x2="-93.98" y2="375.285" width="0.1524" layer="91"/>
+<wire x1="-93.98" y1="375.285" x2="-93.98" y2="379.73" width="0.1524" layer="91"/>
+</segment>
+</net>
